File: hardware/kicad v1 presque fini/untitled.kicad_sch (KiCad schematic)
At the start: 45 parts, among them IC2 L7981TR, IC3 L7981TR, J10 connecteur servo, J11 connecteur uart, J3 connecteur gps, J4 connecteur radio, J5 connecteur servo, J6 reste, J7 connecteur swd, J8 connecteur servo, J9 connecteur servo

Commit message: fin pcb
Parts:
- removed C33: 100n, symbol Device:C_Small
- removed J10, J5, J9: connecteur servo, symbol Connector:Conn_01x03_Pin
- removed J6: reste, symbol Connector:Conn_01x08_Pin
- removed LED1, LED2, LED3, LED4: 587-1024-147F, 5871024147F, symbol ledadressable2020:587-1024-147F
- added IC4: TSC102IDT, SOIC127P600X175-8N, symbol tsc102:TSC102IDT
- added J5: connecteur uart, Connector_JST:JST_SH_BM04B-SRSS-TB_1x04-1MP_P1.00mm_Vertical, symbol Connector:Conn_01x04_Pin
- added R21: 20k, Resistor_SMD:R_0402_1005Metric_Pad0.72x0.64mm_HandSolder, symbol Device:R_Small
- added R22: 10k, Resistor_SMD:R_0402_1005Metric_Pad0.72x0.64mm_HandSolder, symbol Device:R_Small
- added R23: 10m, symbol Device:R_Small
- added R24: 100R, Resistor_SMD:R_0402_1005Metric_Pad0.72x0.64mm_HandSolder, symbol Device:R_Small
- added R25: 2k, Resistor_SMD:R_0402_1005Metric_Pad0.72x0.64mm_HandSolder, symbol Device:R_Small
- added R26: 1k, Resistor_SMD:R_0402_1005Metric_Pad0.72x0.64mm_HandSolder, symbol Device:R_Small
- C18, C19, C20, C22, C25, C26, C27, C28, C30: footprint (none) -> Capacitor_SMD:C_0402_1005Metric_Pad0.74x0.62mm_HandSolder
- C31: value 100n -> 1u; footprint (none) -> Capacitor_SMD:C_0402_1005Metric_Pad0.74x0.62mm_HandSolder
- C32: value 100n -> 10n; footprint (none) -> Capacitor_SMD:C_0402_1005Metric_Pad0.74x0.62mm_HandSolder
- J11, J3: footprint (none) -> Connector_JST:JST_SH_BM04B-SRSS-TB_1x04-1MP_P1.00mm_Vertical
- J4, J7: footprint (none) -> Connector_JST:JST_SH_BM06B-SRSS-TB_1x06-1MP_P1.00mm_Vertical
- J8: footprint (none) -> Connector_JST:JST_SH_BM03B-SRSS-TB_1x03-1MP_P1.00mm_Vertical
- R1, R11, R12, R13, R14, R15, R16, R17, R18, R19: footprint (none) -> Resistor_SMD:R_0402_1005Metric_Pad0.72x0.64mm_HandSolder
Connections:
- net TIM1_CH2_PWM5 is gone; now on net TIM3_CHI_PWM4: J8.3 (Pin_3)
- net +3.3V: now also J11.1 (Pin_1), J5.2 (Pin_2); no longer C30.1, C31.1, C32.1
- net +5V: now also C31.1, IC4.6 (VCC), J5.4 (Pin_4)
- net DAC1_OUT1: now also J5.3 (Pin_3)
- net GND: now also C30.1, C32.1, IC4.2 (GND), J5.1 (Pin_1), R22.1, R26.1; no longer C30.2, C32.2
- net VIN: now also IC4.1 (VM), R21.2, R23.1
- new net: IC4.7 (A3), R25.1, R26.2
- new net: IC4.5 (OUT), R24.2, R25.2
- new net: IC4.3 (A1), IC4.4 (A2)
- new net ADC1_IN2_CURR: C32.2, R24.1
- new net ADC1_IN3_VBAT: C30.2, R21.1, R22.2
- new net BAT+: IC4.8 (VP), R23.2
- no-connect marks 3 -> 2
Other:
- note added: "0.16w de dissipation à 4A"
- note added: "60 de gain tot"
- moved on the sheet: J11
