File: hardware/kicad v1 presque fini/untitled.kicad_sch (KiCad schematic)
At the start: 38 parts, among them IC2 LDO40LPU33RY, IC3 L7981TR, IC4 TSC102IDT, IC5 LDO40LPU33RY, J11 connecteur uart, J3 connecteur gps, J4 connecteur radio, J5 connecteur uart, J7 connecteur swd, J8 connecteur servo

Commit message: pcb
Parts:
- removed J11, J5: connecteur uart, Connector_JST:JST_SH_BM04B-SRSS-TB_1x04-1MP_P1.00mm_Vertical, symbol Connector:Conn_01x04_Pin
- removed J4: connecteur radio, Connector_JST:JST_SH_BM06B-SRSS-TB_1x06-1MP_P1.00mm_Vertical, symbol Connector:Conn_01x06_Pin
- removed J7: connecteur swd, Connector_JST:JST_SH_BM06B-SRSS-TB_1x06-1MP_P1.00mm_Vertical, symbol Connector:Conn_01x06_Pin
- removed J8: connecteur servo, Connector_JST:JST_SH_BM03B-SRSS-TB_1x03-1MP_P1.00mm_Vertical, symbol Connector:Conn_01x03_Pin
- added J4: connecteur radio, Connector_JST:JST_SH_BM04B-SRSS-TB_1x04-1MP_P1.00mm_Vertical, symbol Connector:Conn_01x04_Pin
Connections:
- net 3.3VEN: now also J4.1 (Pin_1)
- net GND: now also J4.2 (Pin_2)
- net LPUART1_RX_RADIO: now also J4.4 (Pin_4)
- net LPUART1_TX_RADIO: now also J4.3 (Pin_3)

Commit message: pcb v1 fini
Parts:
- removed TP1: BAT+, TestPoint:TestPoint_Loop_D1.80mm_Drill1.0mm_Beaded, symbol Connector:TestPoint
- added D1, D4, D5: LED, LED_SMD:LED_0603_1608Metric_Pad1.05x0.95mm_HandSolder, symbol Device:LED
- added R11, R4: 80R, Resistor_SMD:R_0402_1005Metric_Pad0.72x0.64mm_HandSolder, symbol Device:R_Small
- added R3: 200R, Resistor_SMD:R_0402_1005Metric_Pad0.72x0.64mm_HandSolder, symbol Device:R_Small
- IC3: footprint L7981TR:SON50P300X300X100-9N-D -> L7981:SON50P300X300X100-9N-D
- IC4: footprint TSC102IDT:SOIC127P600X175-8N -> TSC102:SOIC127P600X175-8N
- L2: footprint inductance wurth:INDPM7373X340N -> inductancewurth:INDPM7373X340N
Connections:
- net +3.3V: now also D5.2 (A)
- net +5V: now also D1.2 (A)
- net 3.3VEN: now also D4.2 (A)
- net GND: now also R11.1, R3.1, R4.1
- net BAT+: now reaches IC4.8 (VP), R23.2
- new net: D4.1 (K), R4.2
- new net: D1.1 (K), R3.2
- new net: D5.1 (K), R11.2
