File: hardware/kicad v1 presque fini/cansatperso.kicad_pcb (KiCad board)
At the start: 6 copper layers, 21.6 x 24.2 mm, 73 parts, among them IC1 2536030320001, IC2 LDO40LPU33RY, IC3 L7981TR, IC4 TSC102IDT, IC5 LDO40LPU33RY, J1 USB, J11 connecteur uart, J2 47309-2651, J3 connecteur gps, J4 connecteur radio, J5 connecteur uart, J7 connecteur swd, J8 connecteur servo, SW1 RSTBTN, SW2 boot, U1 STM32G431CBUx, U2 USBLC6-2SC6, Y1 Crystal_GND24_Small

Commit message: bj
Parts:
- removed J1: USB, Connector_JST:JST_SH_BM04B-SRSS-TB_1x04-1MP_P1.00mm_Vertical
- removed J11, J5: connecteur uart, Connector_JST:JST_SH_BM04B-SRSS-TB_1x04-1MP_P1.00mm_Vertical
- removed J7: connecteur swd, Connector_JST:JST_SH_BM06B-SRSS-TB_1x06-1MP_P1.00mm_Vertical
- removed J8: connecteur servo, Connector_JST:JST_SH_BM03B-SRSS-TB_1x03-1MP_P1.00mm_Vertical
- J3: moved to F.Cu
- J4: moved to B.Cu
- moved D3 58.6 mm to (127.6, 81.0)
- moved C13 58.6 mm to (113.5, 90.0)
- moved C14 58.6 mm to (113.5, 92.0)
- moved C15 58.6 mm to (113.5, 94.0)
- moved C16 58.6 mm to (113.5, 95.9)
- moved C17 58.6 mm to (113.5, 97.9)
- moved R10 58.6 mm to (127.6, 94.0)
- moved R2 58.6 mm to (124.4, 90.0)
- moved R20 58.6 mm to (127.6, 96.0)
- moved R3 58.6 mm to (124.4, 92.0)
- moved R4 58.6 mm to (124.4, 94.0)
- moved R5 58.6 mm to (124.4, 96.0)
- moved R6 58.6 mm to (124.4, 98.0)
- moved R7 58.6 mm to (124.4, 100.0)
- moved R8 58.6 mm to (127.6, 90.0)
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Other:
- board size 21.6 x 24.2 mm -> 20.9 x 19 mm

Commit message: pcb
Parts:
- removed R3, R4: 5.1k, Resistor_SMD:R_0402_1005Metric_Pad0.72x0.64mm_HandSolder
- J3, R21, R22, R23: moved to B.Cu
- J4: value connecteur radio -> connecteur gps; footprint Connector_JST:JST_SH_BM06B-SRSS-TB_1x06-1MP_P1.00mm_Vertical -> Connector_JST:JST_SH_BM04B-SRSS-TB_1x04-1MP_P1.00mm_Vertical
- moved C32 102.7 mm to (180.7, 79.4), turned to 90 degrees
- moved C31 100.4 mm to (176.8, 74.5), turned to 180 degrees
- moved C30 95.5 mm to (176.1, 83.1), turned to 180 degrees
- moved R23 93.4 mm to (175.1, 78.8), turned to 90 degrees
- moved R1 93.1 mm to (194.6, 91.8)
- moved J2 90.7 mm to (187.3, 74.8), turned to 0 degrees
- moved C19 90.1 mm to (194.6, 87.9), turned to -90 degrees
- moved R25 88.8 mm to (180.7, 74.8), turned to -90 degrees
- moved IC5 88.3 mm to (191.9, 92.3), turned to 180 degrees
- moved R26 88.2 mm to (179.0, 74.2)
- moved R24 87.4 mm to (180.7, 77.1), turned to 90 degrees
- moved C18 85.6 mm to (188.6, 91.4), turned to 0 degrees
- moved IC2 84.8 mm to (192.0, 88.6), turned to 180 degrees
- moved C20 84.4 mm to (192.2, 86.2), turned to 0 degrees
- moved R18 84.3 mm to (189.0, 89.0), turned to 90 degrees
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Connections:
- net Net-(J1-Pin_2) renamed USBD-
- net Net-(J1-Pin_3) renamed USBD+
Routing:
- net SPI1_MISO_SD: track 0.00 -> 23.2 mm, vias 0 -> 2
- net SPI1_MOSI_SD: track 0.00 -> 21.6 mm, vias 0 -> 2
- net SPI1_CS_SD: track 0.00 -> 19.6 mm, vias 0 -> 2
- net SPI1_SCK_SD: track 0.00 -> 18.8 mm, vias 0 -> 2
- net LPUART1_RX_RADIO: track 0.00 -> 16.0 mm, vias 0 -> 2
- net LPUART1_TX_RADIO: track 0.00 -> 15.3 mm, vias 0 -> 2
- net ADC1_IN2_CURR: track 0.00 -> 11.8 mm, vias 0 -> 2
- net ADC1_IN3_VBAT: track 0.00 -> 9.04 mm, vias 0 -> 2
- net Net-(U1-PF0): track 0.00 -> 7.69 mm
- net USART3_RX: track 0.00 -> 7.33 mm
- net Net-(IC4-A3): track 0.00 -> 6.75 mm, vias 0 -> 1
- net Net-(U1-PF1): track 0.00 -> 5.81 mm
- net NRST: track 0.00 -> 5.34 mm
- net Net-(U1-VREF+): track 0.00 -> 4.23 mm
- net I2C3_SDA_ACCEL: track 0.00 -> 3.62 mm, vias 0 -> 2
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- added copper zone on F.Cu, net +3.3V
- added copper zone on In3.Cu, net +3.3V
- added copper zone on In4.Cu, net GND
- added copper zone on F.Cu, net Net-(IC4-OUT)
- removed copper zone on In4.Cu, net +5V
- removed copper zone on B.Cu, net GND
- removed copper zone on F.Cu, net GND
- removed copper zone on In3.Cu, net GND
Other:
- board size 20.9 x 19 mm -> 21.5 x 21.4 mm

Commit message: pcb
Parts:
- moved R23 8.91 mm to (174.7, 87.7)
- moved C20 5.09 mm to (194.6, 90.7), turned to -90 degrees
- moved R21 2.87 mm to (174.5, 84.5), turned to -90 degrees
- moved C24 2.78 mm to (182.1, 91.5), turned to -90 degrees
- moved R17 2.18 mm to (188.9, 86.4)
- moved C27 1.53 mm to (187.5, 86.4)
- moved C25 1.31 mm to (183.5, 88.5)
- moved L2 1.23 mm to (180.1, 78.6)
- moved R15 1.21 mm to (185.7, 88.6)
- moved R1 1.19 mm to (194.6, 92.9)
- moved C15 1.15 mm to (194.2, 76.9), turned to 90 degrees
- moved IC3 1.04 mm to (183.8, 85.9)
- moved R16 0.99 mm to (186.5, 87.0)
- moved C26 0.85 mm to (186.5, 84.7)
- moved R18 0.63 mm to (189.2, 89.7)
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Connections:
- J3 pad MP: (no net) -> GND
- J4 pad MP: (no net) -> GND
Routing:
- net 3.3VEN: track 0.86 -> 18.9 mm, vias 1 -> 5
- net VIN: track 1.84 -> 17.8 mm, vias 1 -> 3
- net +3.3V: track 0.68 -> 14.6 mm, vias 14 -> 18
- net PWEN: track 0.90 -> 11.3 mm, vias 1 -> 2
- net Net-(IC4-VP): track 1.92 -> 11.6 mm, vias 1 -> 2
- net D+: track 1.00 -> 8.03 mm
- net D-: track 0.96 -> 7.28 mm
- net I2C3_SCL_ACCEL: track 2.84 -> 8.60 mm
- net I2C3_SDA_ACCEL: track 3.62 -> 8.68 mm
- net +5V: track 1.81 -> 6.30 mm, vias 3 -> 10
- net Net-(IC3-FSW): track 0.00 -> 1.73 mm
- net GND: track 0.82 -> 2.43 mm
- net SWO: track 0.71 -> 2.31 mm
- net LPUART1_RX_RADIO: track 16.0 -> 17.3 mm
- net Net-(IC4-A1): track 0.00 -> 1.27 mm
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- added copper zone on B.Cu, net +3.3V
- added copper zone on B.Cu, net +5V
- added copper zone on In3.Cu, net +5V
- added copper zone on B.Cu, net 3.3VEN
- added copper zone on B.Cu, net ADC1_IN3_VBAT
- added copper zone on B.Cu, net GND
- added copper zone on F.Cu, net GND
- added copper zone on B.Cu, net Net-(C28-Pad2)
- added copper zone on B.Cu, net Net-(D2-K)
- added copper zone on B.Cu, net Net-(IC3-COMP)
- added copper zone on B.Cu, net Net-(IC3-FB)
- added copper zone on B.Cu, net VIN

Commit message: pcb
Parts:
- added ?: , , F.Cu at (172.7, 85.1)
- added REF**: batpad, connecteur custom:batpad, F.Cu at (173.8, 89.9)
- moved R8 0.32 mm to (184.3, 74.1), turned to 0 degrees
Routing:
- net SDDETECT: track 2.12 -> 16.8 mm
- net USART1_RX_GPS: track 1.04 -> 10.7 mm
- net USART1_TX_GPS: track 0.37 -> 8.88 mm
- net LPUART1_RX_RADIO: track 17.3 -> 18.6 mm
- net +3.3V: track 14.6 -> 15.9 mm, vias 18 -> 19
- net GND: track 2.43 -> 1.64 mm, vias 2 -> 84
- net +5V: vias 10 -> 9
Other:
- board size 21.5 x 21.4 mm -> 23.6 x 21.4 mm

Commit message: pcb v1 fini
Parts:
- added 1: , , F.Cu at (173.1, 74.7)
- added 1: , , F.Cu at (173.1, 90.9)
- added 2: , , F.Cu at (173.1, 76.1)
- added 2: , , F.Cu at (173.1, 92.3)
- added 3: , , F.Cu at (173.1, 77.6)
- added 3: , , F.Cu at (173.1, 93.6)
- added 3: , , B.Cu at (173.1, 93.6)
- added 4: , , F.Cu at (195.7, 84.5)
- added 5: , , F.Cu at (195.7, 83.1)
- added 6: , , F.Cu at (195.7, 81.7)
- added 7: , , F.Cu at (195.7, 80.3)
- added 7: , , B.Cu at (195.7, 80.3)
- added 8: , , F.Cu at (195.7, 78.9)
- added ?: , , F.Cu at (174.5, 93.5)
- added ?: , , B.Cu at (173.1, 73.5)
- added ?: , , B.Cu at (195.7, 83.1)
- added ?: , , B.Cu at (195.7, 84.5)
- added ?: , , B.Cu at (174.5, 93.5)
- added ?: , , B.Cu at (195.7, 78.9)
- added ?: , , B.Cu at (195.7, 81.7)
- added ?: , , B.Cu at (173.1, 89.5)
- added ?: , , B.Cu at (173.1, 92.3)
- added ?: , , F.Cu at (173.1, 73.5)
- added ?: , , F.Cu at (173.1, 89.5)
- added ?: , , F.Cu at (180.0, 92.1)
- added ?: , , B.Cu at (173.1, 90.9)
- added ?: , , B.Cu at (173.1, 76.1)
- added ?: , , B.Cu at (173.1, 77.6)
- added ?: , , B.Cu at (173.1, 74.7)
- added D1: LED, LED_SMD:LED_0603_1608Metric_Pad1.05x0.95mm_HandSolder, B.Cu at (174.6, 74.7)
- added D4: LED, LED_SMD:LED_0603_1608Metric_Pad1.05x0.95mm_HandSolder, B.Cu at (188.2, 93.5)
- added D5: LED, LED_SMD:LED_0603_1608Metric_Pad1.05x0.95mm_HandSolder, B.Cu at (185.4, 90.5)
- added G***: LOGO, logo:logo ensea, B.Cu at (193.4, 74.7)
- added R11: 80R, Resistor_SMD:R_0402_1005Metric_Pad0.72x0.64mm_HandSolder, B.Cu at (184.2, 92.6)
- added R3: 200R, Resistor_SMD:R_0402_1005Metric_Pad0.72x0.64mm_HandSolder, B.Cu at (174.4, 78.2)
- added R4: 80R, Resistor_SMD:R_0402_1005Metric_Pad0.72x0.64mm_HandSolder, B.Cu at (186.0, 93.1)
- added REF**: TestPoint_Pad_1.0x1.0mm, TestPoint:TestPoint_Pad_1.0x1.0mm, F.Cu at (180.0, 93.3)
- added REF**: edge pad, connecteurcustom:edge pad, F.Cu at (195.1, 92.7)
- added REF**1: edge pad, connecteurcustom:edge pad, F.Cu at (195.1, 90.3)
- added REF**2: edge pad, connecteurcustom:edge pad, F.Cu at (195.1, 87.9)
- IC3: footprint L7981TR:SON50P300X300X100-9N-D -> L7981:SON50P300X300X100-9N-D
- IC4: footprint TSC102IDT:SOIC127P600X175-8N -> TSC102:SOIC127P600X175-8N
- J2: footprint microsd:47309-2651 -> molexmicrosd:47309-2651
- J4: value connecteur gps -> connecteur radio
- L2: footprint inductance wurth:INDPM7373X340N -> inductancewurth:INDPM7373X340N
- R20: value 510R -> 80R
- SW1, SW2: footprint kxt3:SW_KXT3 -> KXT3:SW_KXT3
- moved ? 4.40 mm to (172.7, 80.7)
- moved REF** 2.10 mm to (173.8, 87.8)
- moved C21 0.92 mm to (188.6, 92.2)
- moved C18 0.14 mm to (188.6, 91.3)
Connections:
- IC4 pad 8: Net-(IC4-VP) -> BAT+
- J3 pad MP: GND -> (no net)
- J4 pad : GND -> (no net)
- J4 pad MP: GND -> (no net)
- R23 pad 2: Net-(IC4-VP) -> BAT+
- REF** pad 1: VIN -> BAT+
- U1 pad 12: DAC1_OUT1 -> ADC2_IN17
Routing:
- net GPIO_EXTI1: track 0.91 -> 23.1 mm, vias 1 -> 2
- net SWDIO: track 1.45 -> 20.4 mm, vias 1 -> 2
- net SWCLK/I2C1_SDA: track 1.13 -> 19.0 mm, vias 1 -> 2
- net SWO: track 2.31 -> 16.8 mm, vias 1 -> 2
- net USART3_RX: track 7.66 -> 21.3 mm, vias 0 -> 2
- net Net-(IC4-VP): track 11.6 -> 0.00 mm, vias 2 -> 0
- net BAT+: track 0.00 -> 11.6 mm, vias 0 -> 2
- net TIM3_CHI_PWM4: track 0.85 -> 9.35 mm
- net ADC2_IN17: track 0.00 -> 8.36 mm, vias 0 -> 2
- net NRST: track 5.71 -> 13.7 mm, vias 0 -> 2
- net I2C3_SDA_ACCEL: track 8.68 -> 15.6 mm, vias 2 -> 3
- net +3.3V: track 15.9 -> 22.5 mm, vias 19 -> 20
- net USART3_TX: track 0.86 -> 6.76 mm, vias 1 -> 2
- net I2C3_SCL_ACCEL: track 8.60 -> 12.8 mm, vias 2 -> 3
- net SPI1_SCK_SD: track 19.0 -> 22.7 mm
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- added copper zone on F.Cu, net +5V
- added copper zone on B.Cu, net BAT+
- added copper zone on F.Cu, net USBD+
- added copper zone on F.Cu, net USBD-
Other:
- board size 23.6 x 21.4 mm -> 24.9 x 21.4 mm
- board text added: "3.3"
- board text added: "3.3v"
- board text added: "5v"
- board text added: "D+"
- board text added: "D-"
- board text added: "G"
- board text added: "S"
- board text added: "adc"
- board text added: "clk"
- board text added: "dio"
- board text added: "ext1"
- board text added: "gnd"
- board text added: "rst"
- board text added: "rx3"
- board text added: "scl"
- board text added: "sda"
- board text added: "swo"
- board text added: "tx3"
