File: hardware/kicad v1 presque fini/cansatperso.kicad_sch (KiCad schematic)
At the start: 36 parts, among them IC1 2536030320001, J1 USB_C_Receptacle_USB2.0_14P, J2 47309-2651, SW1 RSTBTN, SW2 boot, U1 STM32G431CBUx, U2 USBLC6-2SC6, Y1 Crystal_GND24_Small

Commit message: fin pcb
Parts:
- C1, C11, C12, C13, C15, C16, C17: footprint (none) -> Capacitor_SMD:C_0402_1005Metric_Pad0.74x0.62mm_HandSolder
- D3: footprint (none) -> LED_SMD:LED_0603_1608Metric_Pad1.05x0.95mm_HandSolder
- J1: footprint USB4110_USBC_SMT:USB4110_USBC_SMT -> vraieusbwurth:USBC-WURTH
- R10, R7, R8, R9: footprint (none) -> Resistor_SMD:R_0402_1005Metric_Pad0.72x0.64mm_HandSolder
- SW1, SW2: footprint SW_KXT3:SW_KXT3 -> KXT3:SW_KXT3
Connections:
- net ADC1_IN2_CURR: now reaches U1.9 (PA1)
- net SPI3_CS: no longer names the net of U1.3 (PC14)
- net SPI3_MISO: no longer names the net of U1.42 (PB4)
- net SPI3_MOSI: no longer names the net of U1.43 (PB5)
- net SPI3_SCK: no longer names the net of U1.39 (PC10)
- net TIM1_CH2_PWM5: no longer names the net of U1.31 (PA9)
- net TIM1_CH3_PWM6: no longer names the net of U1.32 (PA10)
- net TIM2_CH3_PWM2 renamed ADC1_IN3_VBAT
- net TIM3_CH3_PWM3: no longer names the net of U1.17 (PB0)
- net TIM4_CH4_PWM7_LED: no longer names the net of U1.47 (PB9)
- net TIM8_CH4N_PWM1: no longer names the net of U1.2 (PC13)
- no-connect marks 12 -> 21
Changed lines of the file:
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@@
 	)
 	(no_connect
+		(at 86.36 106.68)
+	)
+	(no_connect
+		(at 119.38 101.6)
+	)
+	(no_connect
 		(at 289.56 52.07)
 	)
 	(no_connect
+		(at 86.36 127)
+	)
+	(no_connect
 		(at 330.2 182.88)
 	)
@@
 	)
 	(no_connect
+		(at 86.36 116.84)
+	)
+	(no_connect
 		(at 330.2 185.42)
 	)
@@
 	)
 	(no_connect
+		(at 86.36 101.6)
+	)
+	(no_connect
 		(at 86.36 149.86)
 	)
 	(no_connect
+		(at 86.36 109.22)
+	)
+	(no_connect
 		(at 80.01 231.14)
 	)
 	(no_connect
+		(at 86.36 139.7)
+	)
+	(no_connect
 		(at 86.36 154.94)
 	)
@@
 	)
 	(no_connect
+		(at 119.38 104.14)
+	)
+	(no_connect
+		(at 86.36 129.54)
+	)
+	(no_connect
 		(at 312.42 54.61)
 	)
@@
 		)
 	)
-	(global_label "TIM8_CH4N_PWM1"
-		(shape input)
-		(at 86.36 106.68 180)
-		(fields_autoplaced yes)
-		(effects
-			(font
-				(size 1.27 1.27)
-			)
-			(justify right)
-		)
-		(property "Intersheetrefs" "${INTERSHEET_REFS}"
-			(at 66.6835 106.68 0)
-			(effects
-				(font
-					(size 1.27 1.27)
-				)
-				(justify right)
-				(hide yes)
-			)
-		)
-	)
-	(global_label "TIM1_CH2_PWM5"
+	(global_label "ADC1_IN3_VBAT"
 		(shape input)
-		(at 119.38 101.6 0)
+		(at 119.38 83.82 0)
 		(fields_autoplaced yes)
 		(effects
@@
 		)
 		(property "Intersheetrefs" "${INTERSHEET_REFS}"
-			(at 137.726 101.6 0)
+			(at 136.6981 83.82 0)
 			(effects
 				(font
@@
 		)
 	)
-	(global_label "SPI3_SCK"
-		(shape input)
-		(at 86.36 101.6 180)
-		(fields_autoplaced yes)
-		(effects
-			(font
-				(size 1.27 1.27)
-			)
-			(justify right)
-		)
-		(property "Intersheetrefs" "${INTERSHEET_REFS}"
-			(at 74.3639 101.6 0)
-			(effects
-				(font
-					(size 1.27 1.27)
-				)
-				(justify right)
-				(hide yes)
-			)
-		)
-	)
 	(global_label "SWCLK{slash}I2C1_SDA"
 		(shape input)
@@
 		)
 	)
-	(global_label "TIM2_CH3_PWM2"
-		(shape input)
-		(at 119.38 83.82 0)
-		(fields_autoplaced yes)
-		(effects
-			(font
-				(size 1.27 1.27)
-			)
-			(justify left)
-		)
-		(property "Intersheetrefs" "${INTERSHEET_REFS}"
-			(at 137.726 83.82 0)
-			(effects
-				(font
-					(size 1.27 1.27)
-				)
-				(justify left)
-				(hide yes)
-			)
-		)
-	)
-	(global_label "TIM1_CH3_PWM6"
-		(shape input)
-		(at 119.38 104.14 0)
-		(fields_autoplaced yes)
-		(effects
-			(font
-				(size 1.27 1.27)
-			)
-			(justify left)
-		)
-		(property "Intersheetrefs" "${INTERSHEET_REFS}"
-			(at 137.726 104.14 0)
-			(effects
-				(font
-					(size 1.27 1.27)
-				)
-				(justify left)
-				(hide yes)
-			)
-		)
-	)
 	(global_label "SPI1_MISO_SD"
 		(shape input)
@@
 		)
 	)
-	(global_label "SPI3_CS"
-		(shape input)
-		(at 86.36 109.22 180)
-		(fields_autoplaced yes)
-		(effects
-			(font
-				(size 1.27 1.27)
-			)
-			(justify right)
-		)
-		(property "Intersheetrefs" "${INTERSHEET_REFS}"
-			(at 75.6339 109.22 0)
-			(effects
-				(font
-					(size 1.27 1.27)
-				)
-				(justify right)
-				(hide yes)
-			)
-		)
-	)
 	(global_label "SPI1_MISO_SD"
 		(shape input)
@@
 		)
 	)
-	(global_label "SPI3_MOSI"
-		(shape input)
-		(at 86.36 129.54 180)
-		(fields_autoplaced yes)
-		(effects
-			(font
-				(size 1.27 1.27)
-			)
-			(justify right)
-		)
-		(property "Intersheetrefs" "${INTERSHEET_REFS}"
-			(at 73.5172 129.54 0)
-			(effects
-				(font
-					(size 1.27 1.27)
-				)
-				(justify right)
-				(hide yes)
-			)
-		)
-	)
 	(global_label "SDDETECT"
 		(shape input)
@@
 		)
 	)
-	(global_label "TIM4_CH4_PWM7_LED"
-		(shape input)
-		(at 86.36 139.7 180)
-		(fields_autoplaced yes)
-		(effects
-			(font
-				(size 1.27 1.27)
-			)
-			(justify right)
-		)
-		(property "Intersheetrefs" "${INTERSHEET_REFS}"
-			(at 63.5993 139.7 0)
-			(effects
-				(font
-					(size 1.27 1.27)
-				)
-				(justify right)
-				(hide yes)
-			)
-		)
-	)
 	(global_label "NRST"
 		(shape input)
@@
 		)
 	)
-	(global_label "LPUART1_TX_RADIO"
+	(global_label "ADC1_IN2_CURR"
 		(shape input)
-		(at 86.36 144.78 180)
+		(at 119.38 81.28 0)
 		(fields_autoplaced yes)
 		(effects
@@
 				(size 1.27 1.27)
 			)
-			(justify right)
+			(justify left)
 		)
 		(property "Intersheetrefs" "${INTERSHEET_REFS}"
-			(at 65.5343 144.78 0)
+			(at 137.4238 81.28 0)
 			(effects
 				(font
 					(size 1.27 1.27)
 				)
-				(justify right)
+				(justify left)
 				(hide yes)
 			)
 		)
 	)
-	(global_label "SPI3_MISO"
+	(global_label "LPUART1_TX_RADIO"
 		(shape input)
-		(at 86.36 127 180)
+		(at 86.36 144.78 180)
 		(fields_autoplaced yes)
 		(effects
@@
 		)
 		(property "Intersheetrefs" "${INTERSHEET_REFS}"
-			(at 73.5172 127 0)
+			(at 65.5343 144.78 0)
 			(effects
 				(font
@@
 		)
 	)
-	(global_label "TIM3_CH3_PWM3"
-		(shape input)
-		(at 86.36 116.84 180)
-		(fields_autoplaced yes)
-		(effects
-			(font
-				(size 1.27 1.27)
-			)
-			(justify right)
-		)
-		(property "Intersheetrefs" "${INTERSHEET_REFS}"
-			(at 68.014 116.84 0)
-			(effects
-				(font
-					(size 1.27 1.27)
-				)
-				(justify right)
-				(hide yes)
-			)
-		)
-	)
 	(symbol
 		(lib_id "power:GND")
@@
 			)
 		)
-		(property "Footprint" ""
+		(property "Footprint" "Resistor_SMD:R_0402_1005Metric_Pad0.72x0.64mm_HandSolder"
 			(at 309.88 151.13 0)
 			(effects
@@
 			)
 		)
-		(property "Footprint" ""
+		(property "Footprint" "Capacitor_SMD:C_0402_1005Metric_Pad0.74x0.62mm_HandSolder"
 			(at 62.23 87.63 0)
 			(effects
@@
 			)
 		)
-		(property "Footprint" ""
+		(property "Footprint" "Capacitor_SMD:C_0402_1005Metric_Pad0.74x0.62mm_HandSolder"
 			(at 45.72 96.52 0)
 			(effects
@@
 			)
 		)
-		(property "Footprint" "SW_KXT3:SW_KXT3"
+		(property "Footprint" "KXT3:SW_KXT3"
 			(at 33.02 121.92 0)
 			(effects
@@
 			)
 		)
-		(property "Footprint" ""
+		(property "Footprint" "Resistor_SMD:R_0402_1005Metric_Pad0.72x0.64mm_HandSolder"
 			(at 313.69 151.13 0)
 			(effects
@@
 			)
 		)
-		(property "Footprint" "USB4110_USBC_SMT:USB4110_USBC_SMT"
+		(property "Footprint" "vraieusbwurth:USBC-WURTH"
 			(at 71.12 220.98 0)
 			(effects
@@
 			)
 		)
-		(property "Footprint" "SW_KXT3:SW_KXT3"
+		(property "Footprint" "KXT3:SW_KXT3"
 			(at 33.02 73.66 0)
 			(effects
@@
 			)
 		)
-		(property "Footprint" ""
+		(property "Footprint" "Capacitor_SMD:C_0402_1005Metric_Pad0.74x0.62mm_HandSolder"
 			(at 260.35 67.31 0)
 			(effects
@@
 			)
 		)
-		(property "Footprint" ""
+		(property "Footprint" "Resistor_SMD:R_0402_1005Metric_Pad0.72x0.64mm_HandSolder"
 			(at 316.23 49.53 0)
 			(effects
@@
 			)
 		)
-		(property "Footprint" ""
+		(property "Footprint" "Capacitor_SMD:C_0402_1005Metric_Pad0.74x0.62mm_HandSolder"
 			(at 318.77 205.74 0)
 			(effects
@@
 			)
 		)
-		(property "Footprint" ""
+		(property "Footprint" "LED_SMD:LED_0603_1608Metric_Pad1.05x0.95mm_HandSolder"
 			(at 62.23 152.4 0)
 			(effects
@@
 			)
 		)
-		(property "Footprint" ""
+		(property "Footprint" "Capacitor_SMD:C_0402_1005Metric_Pad0.74x0.62mm_HandSolder"
 			(at 270.51 67.31 0)
 			(effects
@@
 			)
 		)
-		(property "Footprint" ""
+		(property "Footprint" "Resistor_SMD:R_0402_1005Metric_Pad0.72x0.64mm_HandSolder"
 			(at 256.54 53.34 0)
 			(effects
@@
 			)
 		)
-		(property "Footprint" ""
+		(property "Footprint" "Capacitor_SMD:C_0402_1005Metric_Pad0.74x0.62mm_HandSolder"
 			(at 72.39 66.04 0)
 			(effects
@@
 			)
 		)
-		(property "Footprint" ""
+		(property "Footprint" "Capacitor_SMD:C_0402_1005Metric_Pad0.74x0.62mm_HandSolder"
 			(at 327.66 205.74 0)
 			(effects

Commit message: hf
Parts:
- removed J1: USB_C_Receptacle_USB2.0_14P, vraieusbwurth:USBC-WURTH, symbol LTC4065:USB_C_Receptacle_USB2.0_16P
- removed R3, R4: 5.1k, Resistor_SMD:R_0402_1005Metric_Pad0.72x0.64mm_HandSolder, symbol Device:R_Small
- added J1: USB, Connector_JST:JST_SH_BM04B-SRSS-TB_1x04-1MP_P1.00mm_Vertical, symbol Connector:Conn_01x04_Pin
- IC1: footprint 2536030320001 -> WSEN-ISDS:2536030320001
- J2: footprint 47309-2651 -> microsd:47309-2651
- SW1, SW2: footprint KXT3:SW_KXT3 -> kxt3:SW_KXT3
- Y1: footprint (none) -> crystalmulticomp:MCSJK7U1200101080B10
Connections:
- net GND: now also Y1.2, Y1.4, J1.4 (Pin_4)
- net at U2.1 (I/O1): now also J1.2 (Pin_2)
- net at U2.3 (I/O2): now also J1.3 (Pin_3)
- net at C13.2: now also U1.5 (PF0), Y1.1; no longer Y1.4
- net at C12.1: now also U1.6 (PF1), Y1.3; no longer Y1.2
- net PWEN: now reaches U1.28 (PB15)
- net vusb renamed +5V
- net +5V: now also J1.1 (Pin_1)
- no-connect marks 21 -> 18
Other:
- moved on the sheet: C12, C13, U2

Commit message: pcb
Parts:
- removed J1: USB, Connector_JST:JST_SH_BM04B-SRSS-TB_1x04-1MP_P1.00mm_Vertical, symbol Connector:Conn_01x04_Pin
Connections:
- net USBD-: now reaches U2.1 (I/O1)
- net USBD+: now reaches U2.3 (I/O2)
Other:
- moved on the sheet: C11

Commit message: pcb v1 fini
Parts:
- J2: footprint microsd:47309-2651 -> molexmicrosd:47309-2651
- R20: value 510R -> 80R
- SW1, SW2: footprint kxt3:SW_KXT3 -> KXT3:SW_KXT3
Connections:
- net DAC1_OUT1 renamed ADC2_IN17
Changed lines of the file:
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@@
 		)
 	)
-	(global_label "DAC1_OUT1"
+	(global_label "ADC2_IN17"
 		(shape input)
 		(at 119.38 88.9 0)
@@
 		)
 		(property "Intersheetrefs" "${INTERSHEET_REFS}"
-			(at 133.009 88.9 0)
+			(at 132.5252 88.9 0)
 			(effects
 				(font
@@
 			)
 		)
-		(property "Footprint" "microsd:47309-2651"
+		(property "Footprint" "molexmicrosd:47309-2651"
 			(at 308.61 146.99 0)
 			(effects
@@
 			)
 		)
-		(property "Footprint" "kxt3:SW_KXT3"
+		(property "Footprint" "KXT3:SW_KXT3"
 			(at 33.02 121.92 0)
 			(effects
@@
 			)
 		)
-		(property "Footprint" "kxt3:SW_KXT3"
+		(property "Footprint" "KXT3:SW_KXT3"
 			(at 33.02 73.66 0)
 			(effects
@@
 			)
 		)
-		(property "Value" "510R"
+		(property "Value" "80R"
 			(at 50.8 149.86 90)
 			(effects
