File: hardware/PCB sensors/Carte sensors/Carte sensors.kicad_pcb (KiCad board)
At the start: 2 copper layers, 77 x 24.2 mm, 24 parts, among them J1 Conn_01x04_Pin, J2 Conn_01x04_Pin, J3 Conn_01x04_Pin, J4 Conn_01x04_Pin, SW1 SW_Push

Commit message: carte sensor
Parts:
- moved J1 1.42 mm to (133.6, 61.9)
- moved D1 1.42 mm to (139.8, 54.5)
- moved D2 1.42 mm to (139.8, 49.7)
- moved R1 1.42 mm to (136.1, 54.5)
- moved R3 1.42 mm to (130.5, 58.6)
- moved R6 1.42 mm to (125.4, 62.5)
- moved C1 1.42 mm to (140.8, 43.2)
- moved R4 1.42 mm to (130.5, 57.4)
- moved R5 1.42 mm to (143.4, 43.2)
- moved SW1 1.42 mm to (130.7, 42.3)
- moved C2 1.42 mm to (104.6, 63.0)
- moved R2 1.42 mm to (136.1, 49.6)
- moved Tarvos1 1.42 mm to (117.3, 35.3)
Routing:
- net (no net): vias 35 -> 0
Other:
- board size 77 x 24.2 mm -> 74.9 x 24.2 mm
- board text added: "GND"
- board text added: "RX"
- board text added: "SCL"
- board text added: "SDA"
- board text added: "TX"
- board text added: "VDD"
