File: Hardware/pcb sensor mathieu/untitled.kicad_sch (KiCad schematic)
At the start: 35 parts, among them IC2 LDO40LPU33RY, IC3 LDO40LPU33RY, IC4 AT7456E, J4 Conn_01x04_Pin, SW3 RSTBTN, SW4 boot, SW5 RSTBTN, U1 STM32L432KCUx, U2 STM32L432KCUx

Commit message: pcb sensor fi,is
Parts:
- removed IC4: AT7456E, AT7456:SOP65P640X120-29N, symbol AT7456:AT7456E
- added C12, C30, C8: 1u, Capacitor_SMD:C_0402_1005Metric_Pad0.74x0.62mm_HandSolder, symbol Device:C_Small
- added C7: 10n, Capacitor_SMD:C_0402_1005Metric_Pad0.74x0.62mm_HandSolder, symbol Device:C_Small
- added C9: 100n, Capacitor_SMD:C_0402_1005Metric_Pad0.74x0.62mm_HandSolder, symbol Device:C_Small
- added H1, H2, H3, H4: MountingHole_Pad, MountingHole:MountingHole_3.2mm_M3_Pad_Via, symbol Mechanical:MountingHole_Pad
- added IC1: TSC102IDT, TSC102:SOIC127P600X175-8N, symbol tsc102:TSC102IDT
- added IC4, IC5: MCP14A0151T-E_CH, driver mosfet:SOT95P270X145-6N, symbol mosfet driver:MCP14A0151T-E_CH
- added J10, J7, J8, J9: Conn_01x03_Pin, Connector_PinHeader_2.54mm:PinHeader_1x03_P2.54mm_Vertical, symbol Connector:Conn_01x03_Pin
- added J5, J6: Conn_01x04_Pin, Connector_JST:JST_SH_SM04B-SRSS-TB_1x04-1MP_P1.00mm_Horizontal, symbol Connector:Conn_01x04_Pin
- added Q1, Q2: BSC0909NS, BSC0909NS:PG-TDSON-8-5, symbol BSC0909NS:BSC0909NS
- added R10, R11: 10m, Resistor_SMD:R_1020_2550Metric_Pad1.33x5.20mm_HandSolder, symbol Device:R_Small
- added R12: 2k, Resistor_SMD:R_0402_1005Metric_Pad0.72x0.64mm_HandSolder, symbol Device:R_Small
- added R13: 1k, Resistor_SMD:R_0402_1005Metric_Pad0.72x0.64mm_HandSolder, symbol Device:R_Small
- added R14: 20k, Resistor_SMD:R_0402_1005Metric_Pad0.72x0.64mm_HandSolder, symbol Device:R_Small
- added R15: 10k, Resistor_SMD:R_0402_1005Metric_Pad0.72x0.64mm_HandSolder, symbol Device:R_Small
- added R20, R22: 40k, Resistor_SMD:R_0402_1005Metric_Pad0.72x0.64mm_HandSolder, symbol Device:R_Small
- added R9: 100R, Resistor_SMD:R_0402_1005Metric_Pad0.72x0.64mm_HandSolder, symbol Device:R_Small
Connections:
- net +5V: now also C12.1, C30.1, C8.1, IC1.6 (VCC), IC4.1 (VDD), IC4.4 (EN), IC5.1 (VDD), IC5.4 (EN), J10.1 (Pin_1), J5.1 (Pin_1), J7.1 (Pin_1), J8.1 (Pin_1), J9.1 (Pin_1)
- net B2: no longer U1.15 (PB1)
- net GND: now also C12.2, C30.2, C7.1, C8.2, C9.1, H2.1, H4.1, IC1.2 (GND), IC4.2 (AGND), IC4.5 (GND), IC5.2 (AGND), IC5.5 (GND), J10.2 (Pin_2), J5.2 (Pin_2), J7.2 (Pin_2), J8.2 (Pin_2), J9.2 (Pin_2), R13.1, R15.1
- net MOSFET2: now reaches U1.12 (PA6)
- net MOSFET2: now also IC5.3 (IN)
- net CH6: now reaches U1.19 (PA9)
- net CH6: now also J6.4 (Pin_4)
- net ALIM renamed MOSFET1
- net MOSFET1: now also IC4.3 (IN)
- net B1 renamed CH5
- net CH5: now also J6.3 (Pin_3)
- new net: IC4.6 (~{OUT}), Q2.4 (G), R20.2
- new net: IC5.6 (~{OUT}), Q1.4 (G), R22.2
- new net: IC1.7 (A3), R12.1, R13.2
- new net: IC1.3 (A1), IC1.4 (A2)
- new net: IC1.5 (OUT), R12.2, R9.2
- new net ADC1_IN2_CURR: C7.2, R9.1
- new net ADC1_IN3_VBAT: C9.2, R14.1, R15.2
- new net BAT+: H3.1, IC1.8 (VP), R10.2, R11.2
- new net CH1: J5.3 (Pin_3), J7.3 (Pin_3)
- new net CH2: J5.4 (Pin_4), J8.3 (Pin_3)
- new net CH3: J6.1 (Pin_1), J9.3 (Pin_3)
- new net CH4: J10.3 (Pin_3), J6.2 (Pin_2)
- new net MOS1IN: Q2.1 (S_1), Q2.2 (S_2), Q2.3 (S_3), R20.1
- new net MOS1OUT: Q2.5 (D_1), Q2.6 (D_2), Q2.7 (D_3), Q2.8 (D_4)
- new net MOS2IN: Q1.1 (S_1), Q1.2 (S_2), Q1.3 (S_3), R22.1
- new net MOS2OUT: Q1.5 (D_1), Q1.6 (D_2), Q1.7 (D_3), Q1.8 (D_4)
- new net VIN: H1.1, IC1.1 (VM), R10.1, R11.1, R14.2
- no-connect marks 30 -> 29
Other:
- note added: "60 de gain tot"
- note added: "adc to ppm"
- note added: "capteur courant"
- note added: "centrale voiture rc"
