File: hardware/pcb sensor mathieu/Carte sensors.kicad_pcb (KiCad board)
At the start: 2 copper layers, 47.9 x 34.9 mm, 88 parts, among them IC1 TSC102IDT, IC2 LDO40LPU33RY, IC3 LDO40LPU33RY, IC4 AT7456E, J1 Conn_01x04_Pin, J2 Conn_01x06, J3 Conn_01x04_Pin, J4 Conn_01x04_Pin, SW1 SW_Push, SW3 RSTBTN, SW4 boot, SW5 RSTBTN, U1 STM32L432KCUx, U2 STM32L432KCUx

Commit message: pcb sensor fi,is
Parts:
- added ?: , , F.Cu at (168.7, 117.9)
- added ?: , , F.Cu at (166.7, 117.9)
- added ?: , , F.Cu at (156.1, 119.2)
- added ?: , , F.Cu at (173.2, 120.7)
- added ?: , , F.Cu at (170.8, 117.9)
- added ?: , , F.Cu at (156.1, 120.7)
- added C12: 1u, Capacitor_SMD:C_0402_1005Metric_Pad0.74x0.62mm_HandSolder, F.Cu at (156.9, 123.9)
- added C30: 1u, Capacitor_SMD:C_0402_1005Metric_Pad0.74x0.62mm_HandSolder, F.Cu at (156.9, 127.6)
- added G***: LOGO, logo:logo ensea, F.Cu at (192.4, 108.3)
- added G***: LOGO, logo:logo ensea, B.Cu at (157.7, 103.3)
- added IC5: MCP14A0151T-E_CH, driver mosfet:SOT95P270X145-6N, F.Cu at (154.1, 126.9)
- added J10: Conn_01x03_Pin, Connector_PinHeader_2.54mm:PinHeader_1x03_P2.54mm_Vertical, F.Cu at (159.8, 135.1)
- added J5: Conn_01x04_Pin, Connector_JST:JST_SH_SM04B-SRSS-TB_1x04-1MP_P1.00mm_Horizontal, F.Cu at (170.5, 133.2)
- added J6: Conn_01x04_Pin, Connector_JST:JST_SH_SM04B-SRSS-TB_1x04-1MP_P1.00mm_Horizontal, F.Cu at (170.5, 125.4)
- added J7: Conn_01x03_Pin, Connector_PinHeader_2.54mm:PinHeader_1x03_P2.54mm_Vertical, F.Cu at (156.1, 135.1)
- added J8: Conn_01x03_Pin, Connector_PinHeader_2.54mm:PinHeader_1x03_P2.54mm_Vertical, F.Cu at (156.2, 131.4)
- added J9: Conn_01x03_Pin, Connector_PinHeader_2.54mm:PinHeader_1x03_P2.54mm_Vertical, F.Cu at (159.8, 131.4)
- added Q1: BSC0909NS, BSC0909NS:PG-TDSON-8-5, B.Cu at (154.3, 126.5)
- added Q2: BSC0909NS, BSC0909NS:PG-TDSON-8-5, B.Cu at (154.2, 120.7)
- added R20: 40k, Resistor_SMD:R_0402_1005Metric_Pad0.72x0.64mm_HandSolder, B.Cu at (150.2, 119.5)
- added R22: 40k, Resistor_SMD:R_0402_1005Metric_Pad0.72x0.64mm_HandSolder, B.Cu at (150.3, 125.2)
- added Tarvos1: ~, tarvosiii:Tarvos III, F.Cu at (163.5, 88.5)
- C1, C13, C14, C15, C16, C17, C2, C26, R1, R16, R2, R3, R4, R5, R6, SW1: moved to B.Cu
- IC4: value AT7456E -> MCP14A0151T-E_CH; footprint AT7456:SOP65P640X120-29N -> driver mosfet:SOT95P270X145-6N
- moved ? 139.5 mm to (204.4, 116.9)
- moved ? 139.3 mm to (205.4, 119.6)
- moved ? 139.3 mm to (207.2, 119.6)
- moved ? 139.3 mm to (215.7, 118.4)
- moved C18 139.3 mm to (205.7, 122.8)
- moved C22 139.3 mm to (209.6, 120.5)
- moved C23 139.3 mm to (209.6, 122.4)
- moved C24 139.3 mm to (209.6, 121.5)
- moved C27 139.3 mm to (213.8, 127.6)
- moved C28 139.3 mm to (209.5, 127.5)
- moved C7 139.3 mm to (219.5, 98.1)
- moved C8 139.3 mm to (211.0, 100.6)
- moved C9 139.3 mm to (214.8, 104.5)
- moved D4 139.3 mm to (208.2, 127.1)
- moved D6 139.3 mm to (215.1, 120.9)
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Connections:
- IC4 pad 1: unconnected-(IC4-N.C._1-Pad1) -> +5V
- IC4 pad 2: unconnected-(IC4-N.C._2-Pad2) -> GND
- IC4 pad 3: unconnected-(IC4-DVDD-Pad3) -> MOSFET1
- IC4 pad 4: unconnected-(IC4-DGND-Pad4) -> +5V
- IC4 pad 5: unconnected-(IC4-CLKIN-Pad5) -> GND
- IC4 pad 6: unconnected-(IC4-XFB-Pad6) -> Net-(IC4-~{OUT})
- J1 pad 3: RX -> TX
- J1 pad 4: TX -> RX
- J1 pad MP: (no net) -> GND
- J2 pad MP: (no net) -> GND
- J3 pad MP: (no net) -> GND
- J4 pad MP: (no net) -> GND
- U1 pad 12: unconnected-(U1-PA6-Pad12) -> MOSFET2
- U1 pad 15: B2 -> unconnected-(U1-PB1-Pad15)
- U1 pad 18: B1 -> CH5
- U1 pad 19: unconnected-(U1-PA9-Pad19) -> CH6
- U1 pad 7: ALIM -> MOSFET1
Routing:
- net VDD_IO: track 32.4 -> 79.3 mm, vias 9 -> 17
- net +5V: track 7.65 -> 42.3 mm
- net CH2: track 0.00 -> 18.7 mm
- net CH1: track 0.00 -> 18.4 mm
- net Net-(Tarvos1-UTXD): track 0.00 -> 10.8 mm, vias 0 -> 1
- net CH4: track 0.00 -> 10.7 mm, vias 0 -> 1
- net Net-(Tarvos1-URXD): track 0.00 -> 9.24 mm, vias 0 -> 1
- net MOSFET2: track 0.00 -> 8.00 mm
- net Net-(IC4-~{OUT}): track 0.00 -> 7.53 mm, vias 0 -> 1
- net LPRX: track 0.00 -> 7.44 mm, vias 0 -> 2
- net SWDIO: track 3.57 -> 10.8 mm
- net SCL_P: track 15.3 -> 22.0 mm
- net SDA_P: track 14.6 -> 21.3 mm, vias 3 -> 2
- net Net-(D1-A): track 0.00 -> 6.28 mm, vias 0 -> 1
- net CH3: track 0.00 -> 6.01 mm
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- added copper zone on B.Cu, net +5V
- added copper zone on B.Cu, net CH5
- added copper zone on B.Cu, net CH6
- added copper zone on B.Cu, net LPRX
- added copper zone on B.Cu, net LPTX
- added copper zone on B.Cu, net MOS1IN
- added copper zone on F.Cu, net MOS1IN
- added copper zone on B.Cu, net MOS1OUT
- added copper zone on F.Cu, net MOS1OUT
- added copper zone on B.Cu, net MOS2IN
- added copper zone on F.Cu, net MOS2IN
- added copper zone on B.Cu, net MOS2OUT
- added copper zone on F.Cu, net MOS2OUT
- added copper zone on B.Cu, net Net-(Tarvos1-MODE_1)
Other:
- board size 47.9 x 34.9 mm -> 82.3 x 43.4 mm
- board text added: "3.3v"
- board text added: "5v"
- board text added: "VIN"
- board text added: "VOUT"
- board text added: "adc"
- board text added: "capteur in"
- board text added: "capteur out"
- board text added: "ch1"
- board text added: "ch2"
- board text added: "ch3"
- board text added: "ch4"
- board text added: "curr"
- board text added: "gnd"
- board text added: "mode_1"
- board text added: "mos1in"
- board text added: "mos1out"
- board text added: "mos2in"
- board text added: "mos2out"
- board text added: "nrst"
- board text added: "nrst 3.3v"
- board text added: "swclk"
- board text added: "swdio"
- board text added: "swo"
- board text added: "tim1ch2"
- board text added: "tim2ch1"
- board text added: "to connect uart to ch5/ch6"
- board text added: "vbat"
