File: hardware/pcb sensor mathieu/Carte sensors.kicad_sch (KiCad schematic)
At the start: 42 parts, among them IC1 TSC102IDT, J1 Conn_01x04_Pin, J2 Conn_01x06, J3 Conn_01x04_Pin, SW1 SW_Push

Commit message: pcb
Parts:
- SW1: footprint KXT3:SW_KXT3 -> kxt3:SW_KXT3
Other:
- added sheet carte mathieu (untitled.kicad_sch)
Changed lines of the file:
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@@
 			)
 		)
-		(property "Footprint" "KXT3:SW_KXT3"
+		(property "Footprint" "kxt3:SW_KXT3"
 			(at 180.34 26.416 0)
 			(effects
@@
 				)
 			)
+		)
+	)
+	(sheet
+		(at 238.76 148.336)
+		(size 21.844 8.89)
+		(fields_autoplaced yes)
+		(stroke
+			(width 0.1524)
+			(type solid)
+		)
+		(fill
+			(color 0 0 0 0.0000)
+		)
+		(property "Sheetname" "carte mathieu"
+			(at 238.76 147.6244 0)
+			(effects
+				(font
+					(size 1.27 1.27)
+				)
+				(justify left bottom)
+			)
+		)
+		(property "Sheetfile" "untitled.kicad_sch"
+			(at 238.76 157.8106 0)
+			(effects
+				(font
+					(size 1.27 1.27)
+				)
+				(justify left top)
+			)
+		)
+		(instances
+			(project "Carte sensors"
+				(path "/bbf03fb3-1189-4874-b08b-8de2caec58f5"
+					(page "2")
+				)
+			)

Commit message: pcb
Parts:
- Tarvos1: footprint Tarvos III:Tarvos III -> tarvosiii:Tarvos III
Changed lines of the file:
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@@
 			)
 		)
-		(property "Footprint" "Tarvos III:Tarvos III"
+		(property "Footprint" "tarvosiii:Tarvos III"
 			(at 141.986 17.78 0)
 			(effects

Commit message: pcb sensor fi,is
Parts:
- removed C7: 10n, Capacitor_SMD:C_0402_1005Metric_Pad0.74x0.62mm_HandSolder, symbol Device:C_Small
- removed C8: 1u, Capacitor_SMD:C_0402_1005Metric_Pad0.74x0.62mm_HandSolder, symbol Device:C_Small
- removed C9: 100n, Capacitor_SMD:C_0402_1005Metric_Pad0.74x0.62mm_HandSolder, symbol Device:C_Small
- removed H1, H2, H3, H4: MountingHole_Pad, MountingHole:MountingHole_3.2mm_M3_Pad_Via, symbol Mechanical:MountingHole_Pad
- removed IC1: TSC102IDT, TSC102:SOIC127P600X175-8N, symbol tsc102:TSC102IDT
- removed R10, R15: 10m, Resistor_SMD:R_1020_2550Metric_Pad1.33x5.20mm_HandSolder, symbol Device:R_Small
- removed R11: 2k, Resistor_SMD:R_0402_1005Metric_Pad0.72x0.64mm_HandSolder, symbol Device:R_Small
- removed R12: 1k, Resistor_SMD:R_0402_1005Metric_Pad0.72x0.64mm_HandSolder, symbol Device:R_Small
- removed R13: 20k, Resistor_SMD:R_0402_1005Metric_Pad0.72x0.64mm_HandSolder, symbol Device:R_Small
- removed R14: 10k, Resistor_SMD:R_0402_1005Metric_Pad0.72x0.64mm_HandSolder, symbol Device:R_Small
- removed R9: 100R, Resistor_SMD:R_0402_1005Metric_Pad0.72x0.64mm_HandSolder, symbol Device:R_Small
Connections:
- net RX: now also J1.4 (Pin_4); no longer J1.3 (Pin_3)
- net TX: now also J1.3 (Pin_3); no longer J1.4 (Pin_4)
Other:
- note added: "I2C et barometre"
- note removed: "60 de gain tot"
- note removed: "I2C"
