File: Hardware/PCB/pcb sensor mathieu/Carte sensors.kicad_pcb (KiCad board)
At the start: 2 copper layers, 82.3 x 43.4 mm, 110 parts, among them IC1 TSC102IDT, IC2 LDO40LPU33RY, IC3 LDO40LPU33RY, IC4 MCP14A0151T-E_CH, IC5 MCP14A0151T-E_CH, J1 Conn_01x04_Pin, J10 Conn_01x03_Pin, J2 Conn_01x06, J3 Conn_01x04_Pin, J4 Conn_01x04_Pin, J5 Conn_01x04_Pin, J6 Conn_01x04_Pin, J7 Conn_01x03_Pin, J8 Conn_01x03_Pin, J9 Conn_01x03_Pin, Q1 BSC0909NS, Q2 BSC0909NS, SW1 SW_Push, SW3 RSTBTN, SW4 boot, SW5 RSTBTN, U1 STM32L432KCUx, U2 STM32L432KCUx

Commit message: carte mathieu
Parts:
- added ?: , , B.Cu at (204.8, 128.0)
- added C29: 10n, Capacitor_SMD:C_0402_1005Metric_Pad0.74x0.62mm_HandSolder, B.Cu at (212.8, 126.3)
- added R23: 10k, Resistor_SMD:R_0402_1005Metric_Pad0.72x0.64mm_HandSolder, B.Cu at (211.8, 126.4)
- added R26: 10k, Resistor_SMD:R_0402_1005Metric_Pad0.72x0.64mm_HandSolder, B.Cu at (213.8, 126.4)
- added SW2: Boutton 2, kxt3:SW_KXT3, B.Cu at (214.5, 128.5)
- R17, R18, R3, R4: value 1000 -> 1k
Connections:
- J4 pad 2: ADC1_IN9 -> OLED_SCL
- J4 pad 3: ADC1_IN10 -> OLED_SDA
- U2 pad 13: unconnected-(U2-PA7-Pad13) -> OLED_SCL
- U2 pad 27: unconnected-(U2-PB4-Pad27) -> OLED_SDA
Routing:
- net OLED_SDA: track 0.00 -> 9.47 mm, vias 0 -> 1
- net OLED_SCL: track 0.00 -> 5.50 mm, vias 0 -> 1
- net Net-(R23-Pad2): track 0.00 -> 5.16 mm
- net ADC1_IN10: track 4.12 -> 0.00 mm, vias 1 -> 0
- net ADC1_IN9: track 3.18 -> 7.03 mm
- net B2: track 0.00 -> 2.37 mm, vias 0 -> 1
- net VDD_IO: track 79.3 -> 81.0 mm
- net GND: vias 376 -> 387
Other:
- board text added: "i2c"
- board text added: "mode_1: push to transparent mode"
- board text removed: "mode_1"
