File: Hardware/PCB/pcb sensor mathieu/untitled.kicad_sch (KiCad schematic)
At the start: 63 parts, among them IC1 TSC102IDT, IC2 LDO40LPU33RY, IC3 LDO40LPU33RY, IC4 MCP14A0151T-E_CH, IC5 MCP14A0151T-E_CH, J10 Conn_01x03_Pin, J4 Conn_01x04_Pin, J5 Conn_01x04_Pin, J6 Conn_01x04_Pin, J7 Conn_01x03_Pin, J8 Conn_01x03_Pin, J9 Conn_01x03_Pin, Q1 BSC0909NS, Q2 BSC0909NS, SW3 RSTBTN, SW4 boot, SW5 RSTBTN, U1 STM32L432KCUx, U2 STM32L432KCUx

Commit message: carte mathieu
Parts:
- added C29: 10n, Capacitor_SMD:C_0402_1005Metric_Pad0.74x0.62mm_HandSolder, symbol Device:C_Small
- added R23, R26: 10k, Resistor_SMD:R_0402_1005Metric_Pad0.72x0.64mm_HandSolder, symbol Device:R_Small
- added SW2: Boutton 2, kxt3:SW_KXT3, symbol Switch:SW_Push
Connections:
- net +3.3V: now also R23.1
- net ADC1_IN10: no longer J4.3 (Pin_3)
- net ADC1_IN9: no longer J4.2 (Pin_2)
- net B2: now also C29.1, R26.2
- net GND: now also C29.2, SW2.1
- net OLED_SCL: now reaches U2.13 (PA7)
- net OLED_SCL: now also J4.2 (Pin_2)
- net OLED_SDA: now reaches U2.27 (PB4)
- net OLED_SDA: now also J4.3 (Pin_3)
- new net: R23.2, R26.1, SW2.2
- no-connect marks 29 -> 27
Other:
- moved on the sheet: C27, C28, D4, IC3, R25
