File: Hardware/PCB/MAINBOARD/cansatperso.kicad_sch (KiCad schematic)
At the start: 33 parts, among them IC1 2536030320001, J2 47309-2651, SW1 RSTBTN, SW2 boot, U1 STM32G431CBUx, U2 USBLC6-2SC6, Y1 Crystal_GND24_Small

Commit message: Question
Manque pas un 100nF au VDD_IO de l'accel ?
Other:
- note added: "Pk tu mets pas un 100nF de découplage ici ?"
Changed lines of the file:
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@@
+		)
+	)
+	(polyline
+		(pts
+			(xy 293.37 207.01) (xy 293.37 210.82)
+		)
+		(stroke
+			(width 0)
+			(type default)
 		)
 	)
@@
 		(effects
 			(font
+				(size 1.27 1.27)
+			)
+		)
+	)
+	(text "Pk tu mets pas un 100nF de découplage ici ?"
+		(exclude_from_sim no)
+		(at 287.782 214.122 0)
+		(effects
+			(font
