File: Hardware/PCB/MAINBOARD/untitled.kicad_sch (KiCad schematic)
At the start: 39 parts, among them IC2 LDO40LPU33RY, IC3 L7981TR, IC4 TSC102IDT, IC5 LDO40LPU33RY, J3 connecteur gps, J4 connecteur radio

Commit message: debut code principal
Parts:
- R18: value 4.99k -> 8.2k
- R19: value 680R -> 1.1k
Changed lines of the file:
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@@
 			)
 		)
-		(property "Value" "4.99k"
+		(property "Value" "8.2k"
 			(at 259.08 44.4499 0)
 			(effects
@@
 			)
 		)
-		(property "Value" "680R"
+		(property "Value" "1.1k"
 			(at 259.08 57.1499 0)
 			(effects
