File: Hardware/PCB/MAINBOARD v2/pcb/cansatperso.kicad_sch (KiCad schematic)
At the start: 39 parts, among them IC1 2536030320001, J2 47309-2651, SW1 RSTBTN, U1 STM32G431CBUx, U3 BMP581, Y1 Crystal_GND24_Small

Commit message: pcbv2
Parts:
- added R2: 10k, Resistor_SMD:R_0402_1005Metric_Pad0.72x0.64mm_HandSolder, symbol Device:R_Small
Connections:
- net USART3_TX is gone; now on net LPUART1_RX_RADIO: U1.22 (PB10)
- net +3.3V: now also R2.1
- net LPUART1_RX_RADIO: no longer U1.11 (PA3)
- net at IC1.1 (SAO): now also R2.2
- net ADC1_IN1: no longer names the net of U1.8 (PA0)
- net ADC1_IN2_CURR: no longer names the net of U1.9 (PA1)
- net D+: no longer names the net of U1.34 (PA12)
- net D-: no longer names the net of U1.33 (PA11)
- new net EXTI3/PWMONTIM4: U1.11 (PA3)
- no-connect marks 16 -> 19
Other:
- note added: "Attention !!!!!! SAO en HIGH"
- note removed: "Pk tu mets pas un 100nF de découplage ici ?"
