File: Hardware/PCB/MAINBOARD v2/pcb/untitled.kicad_sch (KiCad schematic)
At the start: 42 parts, among them IC2 LDO40LPU33RY, IC3 L7981TR, IC5 LDO40LPU33RY, J1 battery connector, J3 BM03B-SRSS-TB, J4 503548-1022, J5 503548-1222

Commit message: pcb
Parts:
- removed J3: BM03B-SRSS-TB, Connector_JST:JST_SH_BM03B-SRSS-TB_1x03-1MP_P1.00mm_Vertical, symbol sm03B:BM03B-SRSS-TB
- added U2: ~, Connector_JST:JST_SH_BM03B-SRSS-TB_1x03-1MP_P1.00mm_Vertical, symbol jst_librairie:bm03b
- H1, H2, H3, H4: footprint customhole:mountinghole1.2mm -> custom hole:mountinghole1.2mm
- IC2, IC5: footprint LDO40PURY:SON95P300X300X90-7N-D -> ldo40pury:SON95P300X300X90-7N-D
- IC3: footprint L7981:SON50P300X300X100-9N-D -> l7981:SON50P300X300X100-9N-D
- L2: footprint inductancewurth:INDPM7373X340N -> inductance wurth:INDPM7373X340N
Connections:
- net +5V: now also U2.2
- net GND: now also U2.1, U2.MP
- net TIM3_CHI_PWM4: now also U2.3
