File: Hardware/PCB/MAINBOARD v2/pcb/cansatperso.kicad_pcb (KiCad board)
At the start: 6 copper layers, 28.4 x 27 mm, 104 parts, among them IC1 2536030320001, IC2 LDO40LPU33RY, IC3 L7981TR, IC5 LDO40LPU33RY, J1 battery connector, J2 47309-2651, J3 BM03B-SRSS-TB, J4 503548-1022, J5 503548-1222, SW1 RSTBTN, U1 STM32G431CBUx, U3 BMP581, Y1 Crystal_GND24_Small

Commit message: pcb
Parts:
- removed the G*** at (192.5, 84.1)
- removed the REF** at (180.0, 93.4)
- added ?: , , F.Cu at (180.0, 93.3)
- added ANT1: 74889302450, antennesmd:74889302450, F.Cu at (143.5, 75.3)
- added BT1: ML414S, MS414:MS421R-IV03E, F.Cu at (162.5, 84.0)
- added C1: 4.7u, Capacitor_SMD:C_0402_1005Metric, F.Cu at (148.4, 84.0)
- added C10: 1u, Capacitor_SMD:C_0402_1005Metric, B.Cu at (164.4, 88.5)
- added C11: 100n, Capacitor_SMD:C_0402_1005Metric, B.Cu at (165.8, 89.0)
- added C12: 4.7u, Capacitor_SMD:C_0402_1005Metric, B.Cu at (151.9, 81.4)
- added C13: 100n, Capacitor_SMD:C_0402_1005Metric, B.Cu at (150.0, 81.5)
- added C14: 100n, Capacitor_SMD:C_0402_1005Metric, B.Cu at (155.0, 83.1)
- added C15: 10n, Capacitor_SMD:C_0402_1005Metric, F.Cu at (158.9, 82.7)
- added C16: 1u, Capacitor_SMD:C_0402_1005Metric, F.Cu at (158.9, 83.7)
- added C17: 0.1u, Capacitor_SMD:C_0402_1005Metric, F.Cu at (160.3, 81.4)
- added C18: 10n, Capacitor_SMD:C_0402_1005Metric, F.Cu at (158.4, 86.1)
- added C19: 100n, Capacitor_SMD:C_0402_1005Metric, B.Cu at (155.0, 84.1)
- added C2: 100n, Capacitor_SMD:C_0402_1005Metric, B.Cu at (153.0, 88.3)
- added C21: 100n, Capacitor_SMD:C_0402_1005Metric, F.Cu at (156.4, 89.2)
- added C22: 100n, Capacitor_SMD:C_0402_1005Metric, B.Cu at (149.2, 87.1)
- added C23: 100p, Capacitor_SMD:C_0402_1005Metric, F.Cu at (150.3, 79.4)
- added C24: 4.7u, Capacitor_SMD:C_0402_1005Metric, B.Cu at (148.2, 87.1)
- added C25: 100n, Capacitor_SMD:C_0402_1005Metric, B.Cu at (153.5, 80.2)
- added C26: 100n, Capacitor_SMD:C_0402_1005Metric, F.Cu at (157.4, 89.2)
- added C3: 1u, Capacitor_SMD:C_0402_1005Metric, F.Cu at (159.6, 75.0)
- added C4: 1u, Capacitor_SMD:C_0402_1005Metric, F.Cu at (158.4, 77.0)
- added C5: 1u, Capacitor_SMD:C_0402_1005Metric, F.Cu at (155.0, 78.3)
- added C6: 10n, Capacitor_SMD:C_0402_1005Metric, F.Cu at (158.4, 87.9)
- added C7: 10n, Capacitor_SMD:C_0402_1005Metric, B.Cu at (159.2, 91.1)
- added C8: 1u, Capacitor_SMD:C_0402_1005Metric, F.Cu at (165.4, 78.2)
- added C9: 0.1u, Capacitor_SMD:C_0402_1005Metric, F.Cu at (164.4, 85.1)
- added D1: ~, LED_SMD:LED_0201_0603Metric_Pad0.64x0.40mm_HandSolder, F.Cu at (162.9, 76.6)
- added D2: ~, LED_SMD:LED_0201_0603Metric_Pad0.64x0.40mm_HandSolder, B.Cu at (140.7, 91.2)
- added D3: ~, LED_SMD:LED_0201_0603Metric_Pad0.64x0.40mm_HandSolder, B.Cu at (141.6, 91.1)
- added D4: MMBZ33VB-QBZ, MMBZ33VBQBZ:BC847BQBZ, B.Cu at (152.1, 80.1)
- added D5: MMBZ33VB-QBZ, MMBZ33VBQBZ:BC847BQBZ, B.Cu at (149.5, 80.1)
- added FL1: LFCN-2400D, LFCN2400D:DLF162500LT5028A1, F.Cu at (148.5, 75.2)
- added G***: LOGO, logo ensea:logo ensea, B.Cu at (191.8, 84.1)
- added IC1: MLPF-WB-01E3, MLPFWB01E3:MLPFWB01E3, F.Cu at (152.7, 77.9)
- added IC2: W25Q128JVPIQ_TR, w25q128:SON127P600X500X80-9N-D, F.Cu at (162.5, 88.8)
- added IC3: LDO40LPU33RY, ldo40pury:SON95P300X300X90-7N-D, F.Cu at (155.8, 75.7)
- added J1: SM06B-SRSS-TB, Connector_JST:JST_SH_SM06B-SRSS-TB_1x06-1MP_P1.00mm_Horizontal, B.Cu at (150.9, 76.4)
- added J4: USB_C_Receptacle_USB2.0_14P, USBCWURTH:USBC-WURTH, B.Cu at (142.2, 82.8)
- added L1: 2.2u, Inductor_SMD:L_0805_2012Metric, F.Cu at (147.7, 85.8)
- added L2: 10n, Inductor_SMD:L_0402_1005Metric, F.Cu at (147.0, 84.5)
- added PA1010D1: PA1010D, PA1010D:PA1010D, B.Cu at (155.8, 77.8)
- added Q1: 2N7002K, 2N7002KQBZ:2N7002KQB, F.Cu at (162.8, 77.9)
- added R1: 510R, Resistor_SMD:R_0402_1005Metric, B.Cu at (140.6, 89.2)
- added R10: 10k, Resistor_SMD:R_0402_1005Metric, B.Cu at (161.7, 88.4)
- added R11: 470R, Resistor_SMD:R_0402_1005Metric, F.Cu at (156.9, 78.2)
- added R12: 470R, Resistor_SMD:R_0402_1005Metric, F.Cu at (156.6, 79.2)
- added R13: 10k, Resistor_SMD:R_0402_1005Metric, B.Cu at (159.6, 88.8)
- added R14: 5.1k, Resistor_SMD:R_0402_1005Metric, F.Cu at (143.6, 86.0)
- added R15: 5.1k, Resistor_SMD:R_0402_1005Metric, F.Cu at (143.6, 79.5)
- added R16: 10k, Resistor_SMD:R_0402_1005Metric, F.Cu at (158.8, 84.6)
- added R17: 50k, Resistor_SMD:R_0402_1005Metric, F.Cu at (162.7, 75.2)
- added R18: 50k, Resistor_SMD:R_0402_1005Metric, F.Cu at (163.3, 74.0)
- added R19: 10R, Resistor_SMD:R_0402_1005Metric, B.Cu at (153.8, 82.2)
- added R2: 510R, Resistor_SMD:R_0402_1005Metric, B.Cu at (146.5, 88.2)
- added R20: 2.2k, Resistor_SMD:R_0402_1005Metric, B.Cu at (153.8, 81.2)
- added R22: 10k, Resistor_SMD:R_0402_1005Metric, B.Cu at (150.9, 87.5)
- added R23: 2.2k, Resistor_SMD:R_0402_1005Metric, B.Cu at (153.2, 87.3)
- added R24: 10k, Resistor_SMD:R_0402_1005Metric, B.Cu at (148.9, 85.0)
- added R25: 0R, Resistor_SMD:R_0402_1005Metric, B.Cu at (148.9, 82.5)
- added R3: 20k, Resistor_SMD:R_0402_1005Metric, F.Cu at (160.9, 79.1)
- added R4: 1R, Resistor_SMD:R_0402_1005Metric, F.Cu at (158.5, 74.0)
- added R5: 510R, Resistor_SMD:R_0402_1005Metric, F.Cu at (161.3, 74.0)
- added R6: 470k, Resistor_SMD:R_0402_1005Metric, F.Cu at (163.8, 76.7)
- added R7: 10k, Resistor_SMD:R_0402_1005Metric, B.Cu at (165.6, 91.2)
- added R8: 10k, Resistor_SMD:R_0402_1005Metric, B.Cu at (157.2, 88.5)
- added R9: 10k, Resistor_SMD:R_0402_1005Metric, B.Cu at (158.7, 89.2)
- added REF**: TestPoint_Pad_1.0x1.0mm, custom_testpoint:TestPoint_Pad_1.0x1.0mm, F.Cu at (157.6, 91.4)
- added REF**: TestPoint_Pad_1.0x1.0mm, custom_testpoint:TestPoint_Pad_1.0x1.0mm, F.Cu at (156.1, 91.5)
- added REF**: TestPoint_Pad_1.0x1.0mm, custom_testpoint:TestPoint_Pad_1.0x1.0mm, F.Cu at (154.5, 91.5)
- added S1: PTS845VM20PSMTR4_LFS, pts845:PTS845VM20PSMTR4LFS, B.Cu at (162.3, 90.7)
- added S2: PTS845VM20PSMTR4_LFS, pts845:PTS845VM20PSMTR4LFS, B.Cu at (155.8, 90.7)
- added SW1: Int, SW_PCM:SW_PCM, B.Cu at (155.4, 73.7)
- added SW4: boot, KXT3:SW_KXT3, F.Cu at (159.9, 85.9)
- added SW5: RSTBTN, KXT3:SW_KXT3, F.Cu at (158.0, 78.3)
- added TP1: bat-, TestPoint:TestPoint_THTPad_D1.0mm_Drill0.5mm, F.Cu at (165.3, 74.5)
- added TP2: bat+, TestPoint:TestPoint_THTPad_D1.0mm_Drill0.5mm, F.Cu at (165.2, 76.5)
- added U1: STM32WB55CGUx, Package_DFN_QFN:QFN-48-1EP_7x7mm_P0.5mm_EP5.6x5.6mm, F.Cu at (153.7, 84.0)
- added U2: ~, Connector_JST:JST_SH_BM03B-SRSS-TB_1x03-1MP_P1.00mm_Vertical, F.Cu at (193.3, 91.5)
- added U2: LTC4065AEDC, ltc4065:DFN-6_DC_LIT, F.Cu at (160.9, 77.3)
- added U4: USBLC6-2SC6, Package_TO_SOT_SMD:SOT-23-6, F.Cu at (142.9, 83.1)
- added U5: BMP581, BMP581:BMP581, B.Cu at (152.1, 84.7)
- added Y1: Crystal_GND24, crystal 32Mhz:830069494, F.Cu at (147.4, 80.9)
- D1, D3, D4, D5: footprint LED_SMD:LED_0603_1608Metric_Pad1.05x0.95mm_HandSolder -> custom hole:LED_0603_1608Metric_Pad1.05x0.95mm_HandSolder
- H1, H2, H3, H4: footprint customhole:mountinghole1.2mm -> custom hole:mountinghole1.2mm
- IC1: footprint WSEN-ISDS:2536030320001 -> WSEN ISDS:2536030320001
- IC2, IC5: footprint LDO40PURY:SON95P300X300X90-7N-D -> ldo40pury:SON95P300X300X90-7N-D
- IC3: footprint L7981:SON50P300X300X100-9N-D -> l7981:SON50P300X300X100-9N-D
- J1: footprint Connector_JST:JST_XH_B3B-XH-AM_1x03_P2.50mm_Vertical -> custom hole:JST_XH_B3B-XH-AM_1x03_P2.50mm_Vertical
- J2: footprint molexmicrosd:47309-2651 -> micro sd:47309-2651
- J3: value BM03B-SRSS-TB -> OLED; footprint Connector_JST:JST_SH_BM03B-SRSS-TB_1x03-1MP_P1.00mm_Vertical -> Connector_PinSocket_2.54mm:PinSocket_1x04_P2.54mm_Vertical
- L2: footprint inductancewurth:INDPM7373X340N -> inductance wurth:INDPM7373X340N
- U3: footprint bmp581:BMP581 -> BMP581:BMP581
- Y1: footprint crystalmulticomp:MCSJK7U1200101080B10 -> crystal:MCSJK7U1200101080B10
- moved J3 49.5 mm to (143.8, 90.5), turned to 90 degrees
- moved H1 1.93 mm to (176.4, 95.5)
- moved H2 1.11 mm to (191.2, 95.6)
- moved H4 1.07 mm to (191.1, 71.5)
- moved H3 0.89 mm to (176.4, 71.5)
Connections:
- ? pad 1: ADC2_IN17 -> unconnected-(U1-PA4-Pad12)
- J3 pad 2: +5V -> +3.3V
- J3 pad 3: TIM3_CHI_PWM4 -> OLED_SCL
- U1 pad 12: ADC2_IN17 -> unconnected-(U1-PA4-Pad12)
- U1 pad 46: USART3_RX -> unconnected-(U1-PB8-Pad46)
Routing:
- net vusb: track 0.00 -> 41.8 mm, vias 0 -> 5
- net COMPASSCL: track 0.00 -> 24.2 mm, vias 0 -> 2
- net COMPASSDA: track 0.00 -> 23.2 mm, vias 0 -> 2
- net +3.3V: track 36.3 -> 51.9 mm, vias 25 -> 45
- net unconnected-(U1-PB8-Pad46): track 0.00 -> 15.6 mm, vias 0 -> 2
- net USART3_RX: track 15.6 -> 0.00 mm, vias 2 -> 0
- net OLED_SCL: track 0.00 -> 15.4 mm, vias 0 -> 1
- net D+: track 0.00 -> 14.3 mm, vias 0 -> 2
- net D-: track 0.00 -> 13.9 mm, vias 0 -> 2
- net SPI_MOSi: track 0.00 -> 13.8 mm, vias 0 -> 2
- net USART_RX: track 0.00 -> 13.3 mm, vias 0 -> 2
- net ALIMGPS: track 0.00 -> 12.7 mm, vias 0 -> 2
- net Net-(U1-PB0): track 0.00 -> 12.5 mm, vias 0 -> 2
- net SPI_MISO: track 0.00 -> 11.9 mm, vias 0 -> 2
- net Net-(U1-PA4): track 0.00 -> 11.6 mm, vias 0 -> 2
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- added copper zone on In4.Cu, net +3.3V
- added copper zone on B.Cu, net BAT+
- added copper zone on F.Cu, net BAT+
- added copper zone on In3.Cu, net GND
- added copper zone on B.Cu, net GNDGPS
- added copper zone on F.Cu, net GNDGPS
- added copper zone on F.Cu, net Net-(BT1-+)
- added copper zone on F.Cu, net Net-(IC3-EN)
- added copper zone on F.Cu, net Net-(U1-PH3)
- added copper zone on F.Cu, net vusb
Other:
- board size 28.4 x 27 mm -> 56.8 x 27 mm
- board text added: "mathieu.p"
- board text added: "nrst"
- board text added: "pressure"
- board text added: "swclk"
- board text added: "swdio"

Commit message: g
Parts:
- removed ANT1: 74889302450, antennesmd:74889302450
- removed BT1: ML414S, MS414:MS421R-IV03E
- removed the C1 at (148.4, 84.0)
- removed the C10 at (164.4, 88.5)
- removed the C11 at (165.8, 89.0)
- removed the C12 at (151.9, 81.4)
- removed the C13 at (150.0, 81.5)
- removed the C14 at (155.0, 83.1)
- removed the C15 at (158.9, 82.7)
- removed the C16 at (158.9, 83.7)
- removed the C17 at (160.3, 81.4)
- removed the C18 at (158.4, 86.1)
- removed the C19 at (155.0, 84.1)
- removed the C2 at (153.0, 88.3)
- removed the C21 at (156.4, 89.2)
- removed the C22 at (149.2, 87.1)
- removed the C23 at (150.3, 79.4)
- removed the C24 at (148.2, 87.1)
- removed the C25 at (153.5, 80.2)
- removed the C26 at (157.4, 89.2)
- removed the C3 at (159.6, 75.0)
- removed the C4 at (158.4, 77.0)
- removed the C5 at (155.0, 78.3)
- removed the C6 at (158.4, 87.9)
- removed the C7 at (159.2, 91.1)
- removed the C8 at (165.4, 78.2)
- removed the C9 at (164.4, 85.1)
- removed the D1 at (162.9, 76.6)
- removed the D2 at (140.7, 91.2)
- removed the D3 at (141.6, 91.1)
- removed the D4 at (152.1, 80.1)
- removed the D5 at (149.5, 80.1)
- removed FL1: LFCN-2400D, LFCN2400D:DLF162500LT5028A1
- removed the IC1 at (152.7, 77.9)
- removed the IC2 at (162.5, 88.8)
- removed the IC3 at (155.8, 75.7)
- removed the J1 at (150.9, 76.4)
- removed J3: OLED, Connector_PinSocket_2.54mm:PinSocket_1x04_P2.54mm_Vertical
- removed the J4 at (142.2, 82.8)
- removed L1: 2.2u, Inductor_SMD:L_0805_2012Metric
- removed the L2 at (147.0, 84.5)
- removed PA1010D1: PA1010D, PA1010D:PA1010D
- removed Q1: 2N7002K, 2N7002KQBZ:2N7002KQB
- removed the R1 at (140.6, 89.2)
- removed the R10 at (161.7, 88.4)
- removed the R11 at (156.9, 78.2)
- removed the R12 at (156.6, 79.2)
- removed the R13 at (159.6, 88.8)
- removed the R14 at (143.6, 86.0)
- removed the R15 at (143.6, 79.5)
- removed the R16 at (158.8, 84.6)
- removed the R17 at (162.7, 75.2)
- removed the R18 at (163.3, 74.0)
- removed the R19 at (153.8, 82.2)
- removed the R2 at (146.5, 88.2)
- removed the R20 at (153.8, 81.2)
- removed the R22 at (150.9, 87.5)
- removed the R23 at (153.2, 87.3)
- removed the R24 at (148.9, 85.0)
- removed the R25 at (148.9, 82.5)
- removed the R3 at (160.9, 79.1)
- removed the R4 at (158.5, 74.0)
- removed the R5 at (161.3, 74.0)
- removed the R6 at (163.8, 76.7)
- removed the R7 at (165.6, 91.2)
- removed the R8 at (157.2, 88.5)
- removed the R9 at (158.7, 89.2)
- removed REF** (x3): TestPoint_Pad_1.0x1.0mm, custom_testpoint:TestPoint_Pad_1.0x1.0mm
- removed S1, S2: PTS845VM20PSMTR4_LFS, pts845:PTS845VM20PSMTR4LFS
- removed the SW1 at (155.4, 73.7)
- removed SW4: boot, KXT3:SW_KXT3
- removed SW5: RSTBTN, KXT3:SW_KXT3
- removed TP1: bat-, TestPoint:TestPoint_THTPad_D1.0mm_Drill0.5mm
- removed TP2: bat+, TestPoint:TestPoint_THTPad_D1.0mm_Drill0.5mm
- removed the U1 at (153.7, 84.0)
- removed the U2 at (160.9, 77.3)
- removed U4: USBLC6-2SC6, Package_TO_SOT_SMD:SOT-23-6
- removed U5: BMP581, BMP581:BMP581
- removed the Y1 at (147.4, 80.9)
Routing:
- net vusb: track 41.8 -> 0.00 mm, vias 5 -> 0
- net COMPASSCL: track 24.2 -> 0.00 mm, vias 2 -> 0
- net COMPASSDA: track 23.2 -> 0.00 mm, vias 2 -> 0
- net +3.3V: track 51.9 -> 36.3 mm, vias 45 -> 25
- net OLED_SCL: track 15.4 -> 0.00 mm, vias 1 -> 0
- net D+: track 14.3 -> 0.00 mm, vias 2 -> 0
- net D-: track 13.9 -> 0.00 mm, vias 2 -> 0
- net SPI_MOSi: track 13.8 -> 0.00 mm, vias 2 -> 0
- net USART_RX: track 13.3 -> 0.00 mm, vias 2 -> 0
- net ALIMGPS: track 12.7 -> 0.00 mm, vias 2 -> 0
- net Net-(U1-PB0): track 12.5 -> 0.00 mm, vias 2 -> 0
- net SPI_MISO: track 11.9 -> 0.00 mm, vias 2 -> 0
- net Net-(U1-PA4): track 11.6 -> 0.00 mm, vias 2 -> 0
- net SPI_SCK: track 11.4 -> 0.00 mm, vias 2 -> 0
- net Net-(IC3-EN): track 9.50 -> 0.00 mm, vias 6 -> 0
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- removed copper zone on In4.Cu, net +3.3V
- removed copper zone on B.Cu, net BAT+
- removed copper zone on F.Cu, net BAT+
- removed copper zone on In3.Cu, net GND
- removed copper zone on B.Cu, net GNDGPS
- removed copper zone on F.Cu, net GNDGPS
- removed copper zone on F.Cu, net Net-(BT1-+)
- removed copper zone on F.Cu, net Net-(IC3-EN)
- removed copper zone on F.Cu, net Net-(U1-PH3)
- removed copper zone on F.Cu, net vusb
Other:
- board size 56.8 x 27 mm -> 28.4 x 27 mm
- board text removed: "mathieu.p"
- board text removed: "nrst"
- board text removed: "pressure"
- board text removed: "swclk"
- board text removed: "swdio"
