File: Hardware/PCB/flexpcb(ne pas ptn de toucher)/flexpcb.kicad_pcb (KiCad board)
At the start: 2 copper layers, 25 parts, among them J1 503552-1022, J2 503552-1222, SW1 SW_Push

Commit message: d
Parts:
- added SW2: SW_Push, Button_Switch_SMD:SW_Push_1P1T_NO_CK_PTS125Sx43PSMTR, F.Cu at (215.6, 91.1)
- added U1: ~, Connector_JST:JST_SH_BM06B-SRSS-TB_1x06-1MP_P1.00mm_Vertical, F.Cu at (154.2, 91.9)
- added U2: ~, Connector_JST:JST_SH_BM02B-SRSS-TB_1x02-1MP_P1.00mm_Vertical, F.Cu at (163.1, 91.9)
- R7: value 1k -> 470R
- R8: value 1k -> 470r
- moved PA1010D1 74.9 mm to (189.1, 98.0)
- moved Tarvos1 61.2 mm to (90.4, 52.2)
- moved C1 13.9 mm to (189.3, 60.5)
- moved C2 13.9 mm to (189.3, 62.5)
- moved C3 13.9 mm to (189.3, 64.5)
- moved C4 13.9 mm to (189.3, 66.4)
- moved C6 13.9 mm to (180.5, 82.0)
- moved C7 13.9 mm to (180.5, 84.0)
- moved J1 13.9 mm to (205.1, 73.8)
- moved J2 13.9 mm to (196.7, 75.6)
- moved LED1 13.9 mm to (176.2, 83.9)
- moved LED2 13.9 mm to (176.2, 89.6)
- moved BT1 13.9 mm to (199.5, 65.1)
- moved R4 13.9 mm to (182.9, 61.3)
- moved C5 13.9 mm to (209.2, 65.1)
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Connections:
- J1 pad 10: vin -> EXTI0
