File: Hardware/PCB/flexpcb(ne pas ptn de toucher)/flexpcb.kicad_sch (KiCad schematic)
At the start: 28 parts, among them J1 503552-1022, J2 503552-1222, J3 Conn_01x02_Pin, SW1 SW_Push, SW2 SW_Push

Commit message: d
Parts:
- removed J3: Conn_01x02_Pin, symbol Connector:Conn_01x02_Pin
- added U2: ~, Connector_JST:JST_SH_BM02B-SRSS-TB_1x02-1MP_P1.00mm_Vertical, symbol jst_librairie:bm02B_jst_sh
- LED1, LED2: footprint (none) -> led adressable:5871024147F
- SW2: footprint (none) -> Button_Switch_SMD:SW_Push_1P1T_NO_CK_PTS125Sx43PSMTR
- U1: footprint (none) -> Connector_JST:JST_SH_BM06B-SRSS-TB_1x06-1MP_P1.00mm_Vertical
Connections:
- net +3.3V: now also U2. (MP)
- net GND: now also U2. (MP)
- net exti1: now also U2. (MP)
- net nrst: now also U1. (MP)
- net swclk: now also U1. (MP)
- net swdio: now also U1. (MP)
- net swo: now also U1. (MP)
- no-connect marks 22 -> 23
Other:
- moved on the sheet: U1
