File: Hardware/PCB/MAINBOARD/Projet_timer/Projet_timer.kicad_sch (KiCad schematic)
At the start: 18 parts, among them IC1 AP1509-50SG-13, IC2 TMC6300-LA-T, U1 AP130-33Y, U2 STM32G431C6Tx

Commit message: maj
Parts:
- added U3: MT6701CT, Package_SO:SO-8_3.9x4.9mm_P1.27mm, symbol Sensor_Magnetic:MT6701CT
Changed lines of the file:
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@@
+	)
+	(symbol
+		(lib_id "Sensor_Magnetic:MT6701CT")
+		(at 250.698 46.482 0)
+		(unit 1)
+		(exclude_from_sim no)
+		(in_bom yes)
+		(on_board yes)
+		(dnp no)
+		(fields_autoplaced yes)
+		(property "Reference" "U3"
+			(at 252.8921 26.67 0)
+			(effects
+				(font
+					(size 1.27 1.27)
+				)
+				(justify left)
+			)
+		)
+		(property "Value" "MT6701CT"
+			(at 252.8921 29.21 0)
+			(effects
+				(font
+					(size 1.27 1.27)
+				)
+				(justify left)
+			)
+		)
+		(property "Footprint" "Package_SO:SO-8_3.9x4.9mm_P1.27mm"
+			(at 250.698 76.962 0)
+			(effects
+				(font
+					(size 1.27 1.27)
+				)
+				(hide yes)
+			)
+		)
+		(property "Datasheet" "https://www.magntek.com.cn/upload/MT6701_Rev.1.5.pdf"
+			(at 250.698 79.502 0)
+			(effects
+				(font
+					(size 1.27 1.27)
+				)
+				(hide yes)
+			)
+		)
+		(property "Description" "Hall Based Angle Position Encoder Sensor, I2C, SSI, ABZ & UVW interfaces, 3.3..5V supply, SOIC-8"
+			(at 250.698 46.482 0)
+			(effects
+				(font
+					(size 1.27 1.27)
+				)
+				(hide yes)
+			)
+		)
+		(pin "2"
+		)
+		(pin "1"
+		)
+		(pin "5"
+		)
+		(pin "8"
+		)
+		(pin "4"
+		)
+		(pin "3"
+		)
+		(pin "6"
+		)
+		(pin "7"
+		)
+		(instances
+			(project ""
+				(path "/294d9c00-ce6c-413e-a002-64ea70696540"
+					(reference "U3")
+					(unit 1)
+				)
+			)
+		)
 	)
 	(symbol
