File: Hardware/PCB/flexpcb(ne pas toucher)/flexpcb.kicad_sch (KiCad schematic)
At the start: 28 parts, among them J1 503552-1022, J2 503552-1222, SW1 SW_Push, SW2 SW_Push

Commit message: flexpcb
Parts:
- removed BT1: ML414S, ms414:MS421R-IV03E, symbol Device:Battery
Connections:
- net +3.3V: now also U2.2; no longer U2. (MP)
- net GND: now also U1.5, U1.MP, U2.MP; no longer U1. (MP), U2. (MP)
- net exti1: now also U2.1; no longer U2. (MP)
- net nrst: now also U1.4; no longer U1. (MP)
- net swclk: now also U1.2; no longer U1. (MP)
- net swdio: now also U1.3; no longer U1. (MP)
- net swo: now also U1.1; no longer U1. (MP)
Changed lines of the file:
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@@
 	)
 	(junction
-		(at 93.218 93.726)
-		(diameter 0)
-		(color 0 0 0 0)
-	)
-	(junction
 		(at 83.82 76.2)
 		(diameter 0)
@@
 	)
 	(junction
-		(at 98.806 83.566)
-		(diameter 0)
-		(color 0 0 0 0)
-	)
-	(junction
 		(at 104.648 40.386)
 		(diameter 0)
@@
 	)
 	(no_connect
-		(at 105.41 162.56)
+		(at 107.95 162.56)
 	)
 	(no_connect
@@
 	(wire
 		(pts
+			(xy 107.95 151.13) (xy 105.41 151.13)
+		)
+		(stroke
+			(width 0)
+			(type default)
+		)
+	)
+	(wire
+		(pts
 			(xy 85.344 88.9) (xy 84.074 88.9)
 		)
@@
 	(wire
 		(pts
+			(xy 107.95 147.32) (xy 105.41 147.32)
+		)
+		(stroke
+			(width 0)
+			(type default)
+		)
+	)
+	(wire
+		(pts
 			(xy 49.022 92.456) (xy 49.022 91.44)
 		)
@@
 	(wire
 		(pts
-			(xy 66.04 43.18) (xy 61.722 43.18)
+			(xy 107.95 143.51) (xy 105.41 143.51)
 		)
 		(stroke
@@
 	(wire
 		(pts
-			(xy 104.648 50.038) (xy 104.648 47.752)
+			(xy 66.04 43.18) (xy 61.722 43.18)
 		)
 		(stroke
@@
 	(wire
 		(pts
-			(xy 98.806 83.566) (xy 102.108 83.566)
+			(xy 104.648 50.038) (xy 104.648 47.752)
 		)
 		(stroke
@@
 	(wire
 		(pts
+			(xy 120.65 167.64) (xy 118.11 167.64)
+		)
+		(stroke
+			(width 0)
+			(type default)
+		)
+	)
+	(wire
+		(pts
 			(xy 90.17 35.306) (xy 87.884 35.306)
 		)
@@
 	(wire
 		(pts
-			(xy 93.218 93.726) (xy 102.108 93.726)
+			(xy 83.82 71.882) (xy 83.82 76.2)
 		)
 		(stroke
@@
 	(wire
 		(pts
-			(xy 83.82 71.882) (xy 83.82 76.2)
+			(xy 61.214 33.02) (xy 66.04 33.02)
 		)
 		(stroke
@@
 	(wire
 		(pts
-			(xy 61.214 33.02) (xy 66.04 33.02)
+			(xy 59.944 31.75) (xy 66.04 31.75)
 		)
 		(stroke
@@
 	(wire
 		(pts
-			(xy 59.944 31.75) (xy 66.04 31.75)
+			(xy 66.04 34.29) (xy 61.214 34.29)
 		)
 		(stroke
@@
 	(wire
 		(pts
-			(xy 66.04 34.29) (xy 61.214 34.29)
+			(xy 107.95 158.75) (xy 105.41 158.75)
 		)
 		(stroke
@@
 		)
 	)
+	(wire
+		(pts
+			(xy 107.95 154.94) (xy 105.41 154.94)
+		)
+		(stroke
+			(width 0)
+			(type default)
+		)
+	)
 	(rectangle
 		(start 151.13 27.94)
@@
 	)
 	(symbol
-		(lib_id "Device:Battery")
-		(at 102.108 88.646 0)
-		(unit 1)
-		(exclude_from_sim no)
-		(in_bom yes)
-		(on_board yes)
-		(dnp no)
-		(property "Reference" "BT1"
-			(at 106.426 85.852 0)
-			(effects
-				(font
-					(size 1.27 1.27)
-				)
-				(justify left)
-			)
-		)
-		(property "Value" "ML414S"
-			(at 105.918 89.408 0)
-			(effects
-				(font
-					(size 1.27 1.27)
-				)
-				(justify left)
-			)
-		)
-		(property "Footprint" "ms414:MS421R-IV03E"
-			(at 102.108 87.122 90)
-			(effects
-				(font
-					(size 1.27 1.27)
-				)
-				(hide yes)
-			)
-		)
-		(property "Datasheet" "~"
-			(at 102.108 87.122 90)
-			(effects
-				(font
-					(size 1.27 1.27)
-				)
-				(hide yes)
-			)
-		)
-		(property "Description" "Multiple-cell battery"
-			(at 102.108 88.646 0)
-			(effects
-				(font
-					(size 1.27 1.27)
-				)
-				(hide yes)
-			)
-		)
-		(pin "2"
-		)
-		(pin "1"
-		)
-		(instances
-			(project "flexpcb"
-				(path "/46b50a93-e56b-49e1-bdd2-66a4d6fc6bf5"
-					(reference "BT1")
-					(unit 1)
-				)
-			)
-		)
-	)
-	(symbol
 		(lib_id "power:GND")
 		(at 190.5 55.88 90)
@@
 	(symbol
 		(lib_id "jst_sh_symboles:jst_sh_6pin")
-		(at 116.84 153.67 0)
+		(at 119.38 153.67 0)
 		(unit 1)
 		(exclude_from_sim no)
@@
 		(fields_autoplaced yes)
 		(property "Reference" "U1"
-			(at 123.19 151.7649 0)
+			(at 125.73 151.7649 0)
 			(effects
 				(font
@@
 		)
 		(property "Value" "~"
-			(at 123.19 153.67 0)
+			(at 125.73 153.67 0)
 			(effects
 				(font
@@
 		)
 		(property "Footprint" "Connector_JST:JST_SH_BM06B-SRSS-TB_1x06-1MP_P1.00mm_Vertical"
-			(at 116.84 153.67 0)
+			(at 119.38 153.67 0)
 			(effects
 				(font
@@
 		)
 		(property "Datasheet" ""
-			(at 116.84 153.67 0)
+			(at 119.38 153.67 0)
 			(effects
 				(font
@@
 		)
 		(property "Description" ""
-			(at 116.84 153.67 0)
+			(at 119.38 153.67 0)
 			(effects
 				(font
@@
 			)
 		)
-		(pin ""
+		(pin "MP"
 		)
-		(pin ""
+		(pin "5"
 		)
-		(pin ""
+		(pin "1"
 		)
-		(pin ""
+		(pin "3"
 		)
-		(pin ""
+		(pin "4"
 		)
-		(pin ""
+		(pin "6"
 		)
-		(pin ""
+		(pin "2"
 		)
 		(instances
@@
 			)
 		)
-		(pin ""
+		(pin "2"
 		)
-		(pin ""
+		(pin "MP"
 		)
-		(pin ""
+		(pin "1"
 		)
 		(instances
