File: Hardware/PCB/flexpcb(ne pas toucher)/flexpcb.kicad_pcb (KiCad board)
At the start: 2 copper layers, 28 parts, among them J1 503552-1022, J2 503552-1222, SW1 SW_Push, SW2 SW_Push

Commit message: flexpcb
Parts:
- removed BT1: ML414S, ms414:MS421R-IV03E
- added ?: , , F.Cu at (104.4, 117.2)
- added ?: , , F.Cu at (77.8, 118.5)
- added ?: , , F.Cu at (150.4, 110.4)
- added ?: , , F.Cu at (77.7, 109.3)
- added ?: , , F.Cu at (93.4, 118.2)
- added ?: , , F.Cu at (104.3, 109.5)
- added ?: , , F.Cu at (124.5, 82.9)
- added ?: , , F.Cu at (156.9, 95.4)
- added ?: , , F.Cu at (106.3, 66.0)
- added ?: , , F.Cu at (93.4, 109.0)
- added ?: , , F.Cu at (114.2, 82.9)
- added REF**: mountinghole1.2mm, custom hole:mountinghole1.2mm, F.Cu at (79.5, 87.4)
- C1, C2, C3, C4, C5, C6, C7, D1, D2, LED1, LED2, PA1010D1, R1, R2, R3, R4, R5, R6, R7, R8, SW2, Tarvos1, U1, U2: moved to B.Cu
- moved SW2 132.0 mm to (85.6, 113.6), turned to 90 degrees
- moved D1 123.4 mm to (84.3, 87.9), turned to 180 degrees
- moved D2 119.7 mm to (87.6, 87.8)
- moved C7 108.8 mm to (76.6, 116.4)
- moved C1 107.1 mm to (82.3, 66.5), turned to 180 degrees
- moved LED2 102.4 mm to (76.7, 113.6), turned to 90 degrees
- moved R4 101.4 mm to (84.7, 86.3), turned to 180 degrees
- moved R5 97.9 mm to (87.8, 86.2)
- moved SW1 94.8 mm to (105.9, 84.0), turned to 90 degrees
- moved C2 93.7 mm to (98.6, 86.3), turned to 180 degrees
- moved C6 91.8 mm to (95.5, 116.8), turned to -90 degrees
- moved LED1 86.8 mm to (94.7, 113.5), turned to 180 degrees
- moved R6 82.7 mm to (103.0, 86.4), turned to 180 degrees
- moved R1 79.0 mm to (105.9, 72.8), turned to 90 degrees
- moved R3 78.2 mm to (105.3, 68.7), turned to 90 degrees
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Connections:
- U1 pad 1: (no net) -> swo
- U1 pad 2: (no net) -> swclk
- U1 pad 3: (no net) -> swdio
- U1 pad 4: (no net) -> nrst
- U1 pad 5: (no net) -> GND
- U1 pad 6: (no net) -> unconnected-(U1-Pad6)
- U1 pad MP: (no net) -> GND
- U2 pad 1: (no net) -> exti1
- U2 pad 2: (no net) -> +3.3V
- U2 pad MP: (no net) -> GND
Routing:
- net +3.3V: track 0.00 -> 333.9 mm, vias 0 -> 11
- net TX: track 0.00 -> 88.9 mm, vias 0 -> 1
- net RX: track 0.00 -> 87.1 mm, vias 0 -> 1
- net RX_GPS: track 0.00 -> 79.6 mm, vias 0 -> 1
- net TX_GPS: track 0.00 -> 75.8 mm, vias 0 -> 1
- net EXTI0: track 0.00 -> 75.4 mm, vias 0 -> 4
- net exti1: track 0.00 -> 51.8 mm, vias 0 -> 2
- net exti3/pwmled: track 0.00 -> 47.1 mm, vias 0 -> 1
- net swo: track 0.00 -> 37.4 mm, vias 0 -> 1
- net swclk: track 0.00 -> 36.9 mm, vias 0 -> 1
- net nrst: track 0.00 -> 36.9 mm, vias 0 -> 1
- net swdio: track 0.00 -> 36.6 mm, vias 0 -> 1
- net Net-(Tarvos1-UTXD): track 0.00 -> 23.4 mm
- net Net-(Tarvos1-URXD): track 0.00 -> 22.8 mm
- net Net-(LED1-DOUT): track 0.00 -> 16.9 mm
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- added copper zone on B.Cu, net +3.3V
- added copper zone on B.Cu, net GND
- added copper zone on F.Cu, net GND
Other:
- board outline added: 121.7 x 58.1 mm
- board text added: "ALL zone on USER.eco1 are stiffeners from the exact same size !"
- board text added: "Stiffener on B.cu"
- board text added: "Stiffener on F.cu"
